File: Energy_Meter/Energy_Meter.sch (KiCad schematic (older format))
At the start: 33 parts, among them J1 RJ45, P1 SHUNT, P2 HV, U1 MCP6V27, U2 MAX11644, U3 CRE1S0505S3C, U4 ADUM1250ARZ, U5 MCP2551-I/P, U6 7805, U7 Kitprog-PSoC

Commit message: Energy Meter layout is done
Parts:
- L1, L2: footprint .pretty:13R103C -> Resistors_SMD:R_0805_HandSoldering
- U1, U2: footprint Housings_SOIC:SOIC-8_3.9x4.9mm_Pitch1.27mm -> Housings_SSOP:TSSOP-8_3x3mm_Pitch0.65mm
Changed lines of the file:
@@
 F 0 "U2" H 3050 2900 100 0000 C CNN
 F 1 "MAX11644" H 3050 3050 100 0000 C CNN
-F 2 "Housings_SOIC:SOIC-8_3.9x4.9mm_Pitch1.27mm" H 3050 3350 100 0001 C CNN
+F 2 "Housings_SSOP:TSSOP-8_3x3mm_Pitch0.65mm" H 3050 3350 100 0001 C CNN
 F 3 "" H 3050 3350 100 0000 C CNN
 	1    3050 3350
@@
 F 0 "U1" H 3000 4250 100 0000 C CNN
 F 1 "MCP6V27" H 3000 4400 100 0000 C CNN
-F 2 "Housings_SOIC:SOIC-8_3.9x4.9mm_Pitch1.27mm" H 3000 4700 100 0001 C CNN
+F 2 "Housings_SSOP:TSSOP-8_3x3mm_Pitch0.65mm" H 3000 4700 100 0001 C CNN
 F 3 "" H 3000 4700 100 0000 C CNN
 	1    3000 4700
@@
 F 0 "L1" V 4350 1500 50  0000 C CNN
 F 1 "10uH" V 4500 1500 50  0000 C CNN
-F 2 ".pretty:13R103C" H 4400 1500 50  0001 C CNN
+F 2 "Resistors_SMD:R_0805_HandSoldering" H 4400 1500 50  0001 C CNN
 F 3 "" H 4400 1500 50  0000 C CNN
 	1    4400 1500
@@
 F 0 "L2" V 6750 1500 50  0000 C CNN
 F 1 "10uH" V 6900 1500 50  0000 C CNN
-F 2 ".pretty:13R103C" H 6800 1500 50  0001 C CNN
+F 2 "Resistors_SMD:R_0805_HandSoldering" H 6800 1500 50  0001 C CNN
 F 3 "" H 6800 1500 50  0000 C CNN
 	1    6800 1500

Commit message: Energy Meter is *more* done
Parts:
- removed J1: RJ45, Connect:RJ45_8, symbol RJ45
- added P3: CONN_02X04, Connectors_Molex:Molex_NanoFit_2x04x2.50mm_Straight, symbol CONN_02X04
Connections:
- net +12V: now also P3.5 (P5), P3.6 (P6), P3.7 (P7), P3.8 (P8)
- net CANH: now also P3.1 (P1)
- net CANL: now also P3.4 (P4)
