File: ESF_Diagrams/ESF_Diagrams.sch (KiCad schematic (older format))
At the start: 9 parts

Commit message: CAN bus ESF Diagram
Parts:
- added F1: Main Fuse (800A), symbol Fuse
- added R1, R2: 120, symbol R
- added U1, U4, U5, U6, U7: C-CAN, symbol Generic_CAN_Node
- added U10: AMS, symbol Generic_CAN_Node
- added U8: Raspberry Pi, symbol Generic_CAN_Node
- added U9: Teensy 3.5, symbol Generic_CAN_Node
- BT1: renamed from BT?; value Battery -> 48V
- gave numbers to parts that had none: 8
Connections:
- net at MC1.~ (M-): now also L1.2; no longer M1.~
- net at MC2.~ (M-): now also L2.2; no longer M2.~
- new net: MC1.~ (M-), MC2.~ (M-), U3.~
- new net: F1.1, MC1.~ (M-), MC2.~ (M-)
- new net: M1.~, MC1.~ (M-)
- new net: M2.~, MC2.~ (M-)
- new net: F1.2, U2.~
- new net CANH: R1.1, R2.1, U1.~, U10.~, U4.~, U5.~, U6.~, U7.~, U8.~, U9.~
- new net CANL: R1.2, R2.2, U1.~, U10.~, U4.~, U5.~, U6.~, U7.~, U8.~, U9.~
Other:
- moved on the sheet: BT1, L1, L2, M1, M2, MC1, MC2, U2, U3
