File: ESF_Diagrams/ESF_Diagrams.sch (KiCad schematic (older format))
At the start: 20 parts, among them M1 Motor, M2 Motor, U1 C-CAN, U10 AMS, U2 AIR, U3 AIR, U4 C-CAN, U5 C-CAN, U6 C-CAN, U7 C-CAN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

Commit message: Battery additions
Parts:
- added BT? (x4): Battery_Cell, symbol Battery_Cell
- added BT? (x12): Battery, symbol Battery
Connections:
- net labels added: TS+, TS-
- wire segments 57 -> 122

Commit message: More work on ESF Diagrams
Parts:
- removed U1, U4, U5, U6, U7: C-CAN, symbol Generic_CAN_Node
- removed U10: AMS, symbol Generic_CAN_Node
- removed U8: Raspberry Pi, symbol Generic_CAN_Node
- removed U9: Teensy 3.5, symbol Generic_CAN_Node
- added U?: FL, symbol Generic_CAN_Node
- added U?: FR, symbol Generic_CAN_Node
- added U?: RL, symbol Generic_CAN_Node
- added U?: RR, symbol Generic_CAN_Node
- added U?: PED, symbol Generic_CAN_Node
- added U?: RPi, symbol Generic_CAN_Node
- added U?: VCU, symbol Generic_CAN_Node
- added U?: AMS, symbol Generic_CAN_Node
Connections:
- wire segments 122 -> 87
Other:
- note added: "CAN Bus Architecture"
- moved on the sheet: R1, R2

Commit message: ESF updates, TSAL board updates
Parts:
- added U?: E-Meter, symbol Generic_1x1
Connections:
- wire segments 87 -> 88
Changed lines of the file:
@@
 LIBS:UNCAMotorsports
 LIBS:relays
+LIBS:switches
 LIBS:ESF_Diagrams-cache
 EELAYER 26 0
@@
 U 1 1 585DE2C8
 P 2150 1250
-F 0 "U2" H 2050 1500 60  0000 C CNN
+F 0 "U2" H 2050 1500 60  0001 C CNN
 F 1 "AIR" H 2150 1250 60  0000 C CNN
 F 2 "" H 2150 1250 60  0001 C CNN
@@
 U 1 1 585DEC17
 P 2150 2550
-F 0 "U3" H 2050 2800 60  0000 C CNN
+F 0 "U3" H 2050 2800 60  0001 C CNN
 F 1 "AIR" H 2150 2550 60  0000 C CNN
 F 2 "" H 2150 2550 60  0001 C CNN
@@
 	1600 2550 1750 2550
 Wire Wire Line
-	2550 2550 4350 2550
-Wire Wire Line
 	1600 2550 1600 2100
 Wire Wire Line
@@
 F1 "file5874D542.sch" 60
 $EndSheet
+$Comp
+L Generic_1x1 U?
+U 1 1 58784B31
+P 3250 2550
+F 0 "U?" H 3100 2800 60  0001 C CNN
+F 1 "E-Meter" H 3250 2550 60  0000 C CNN
+F 2 "" H 3250 2550 60  0001 C CNN
+F 3 "" H 3250 2550 60  0001 C CNN
+	1    3250 2550
+	1    0    0    -1
+$EndComp
+Wire Wire Line
+	2850 2550 2550 2550
+Wire Wire Line
+	3650 2550 4350 2550
 $EndSCHEMATC
