File: ESF_Diagrams/file5874D542.sch (KiCad schematic (older format))
At the start: 9 parts

Commit message: Accumulator changes
Connections:
- net at U?.~: now also U?.~; no longer U?.~ (x3)
- new net: U?.~, U?.~ (x2)
Changed lines of the file:
@@
 $Descr A 8500 11000 portrait
 encoding utf-8
-Sheet 2 2
+Sheet 2 3
 Title ""
 Date ""

Commit message: Remake battery drawing
Connections:
- net at U?.~: now also U?.~; no longer U?.~ (x3)
- new net: U?.~, U?.~ (x2)
Changed lines of the file:
@@
 $Descr A 8500 11000 portrait
 encoding utf-8
-Sheet 2 3
+Sheet 2 2
 Title ""
 Date ""
