File: VehicleController/Hardware/VehicleController.sch (KiCad schematic (older format))
At the start: 1 part

Commit message: Create TSAL
Parts:
- removed U?: Teensy_3.2, symbol Teensy_3.2
- added U?: FGMMOPA6H, symbol FGMMOPA6H
- added U?: MS5611, symbol MS5611
- added U?: Teensy_3.5, symbol Teensy_3.5
Changed lines of the file:
@@
 LIBS:contrib
 LIBS:valves
-EELAYER 25 0
+LIBS:VehicleController-cache
+EELAYER 26 0
 EELAYER END
 $Descr A4 11693 8268
@@
 $EndDescr
 $Comp
-L Teensy_3.2 U?
-U 1 1 58252D24
-P 5650 2850
-F 0 "U?" H 4900 4100 60  0000 C CNN
-F 1 "Teensy_3.2" H 6200 1500 60  0000 C CNN
-F 2 "" H 6000 3750 60  0000 C CNN
-F 3 "" H 6000 3750 60  0000 C CNN
-	1    5650 2850
-	-1   0    0    -1
+L FGMMOPA6H U?
+U 1 1 586821A5
+P 1900 2750
+F 0 "U?" H 1950 3437 60  0000 C CNN
+F 1 "FGMMOPA6H" H 1950 3331 60  0000 C CNN
+F 2 "" H 1900 3000 60  0000 C CNN
+F 3 "" H 1900 3000 60  0000 C CNN
+	1    1900 2750
+	1    0    0    -1
+$EndComp
+$Comp
+L MS5611 U?
+U 1 1 58682357
+P 1900 4200
+F 0 "U?" H 1900 4687 60  0000 C CNN
+F 1 "MS5611" H 1900 4581 60  0000 C CNN
+F 2 "" H 1800 4200 60  0000 C CNN
+F 3 "" H 1800 4200 60  0000 C CNN
+	1    1900 4200
+	1    0    0    -1
+$EndComp
+$Comp
+L Teensy_3.5 U?
+U 1 1 586824D0
+P 5400 2350
+F 0 "U?" H 5450 3087 60  0000 C CNN
+F 1 "Teensy_3.5" H 5450 2981 60  0000 C CNN
+F 2 "" H 5400 2350 60  0000 C CNN
+F 3 "" H 5400 2350 60  0000 C CNN
+	1    5400 2350
+	1    0    0    -1
 $EndComp
 $EndSCHEMATC
