File: C-CAN_Y17/C-CAN_Y17.sch (KiCad schematic (older format))
At the start: 29 parts, among them J1 S1_Pull, J2 S2_Pull, J3 S3_Pull, J4 S4_Pull, J5 S5_Pull, P3 CAN_Terminate, P4 MX150_8, P5 MX150_16, SW1 SW_Push, U1 MCP2551-I/SN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

Commit message: C-CAN Fixes
Parts:
- U2: symbol AP1117 -> AP1117-RESCUE-C-CAN_Y17
- U3: footprint UNCAMotorsports:CypressPSoC -> UNCA Motorsports:PSoC5LP
Changed lines of the file:
@@
 EESchema Schematic File Version 2
+LIBS:C-CAN_Y17-rescue
 LIBS:UNCAMotorsports
-LIBS:C-CAN_Y17-rescue
 LIBS:power
 LIBS:device
@@
 F 0 "U3" H 8250 4050 60  0000 C CNN
 F 1 "Cypress_5LP" H 8300 3950 60  0000 C CNN
-F 2 "UNCAMotorsports:CypressPSoC" H 8800 2800 60  0001 C CNN
+F 2 "UNCA Motorsports:PSoC5LP" H 8800 2800 60  0001 C CNN
 F 3 "" H 8800 2800 60  0000 C CNN
 	1    8800 2600
@@
 GND
 $Comp
-L AP1117 U2
+L AP1117-RESCUE-C-CAN_Y17 U2
 U 1 1 58BD7651
 P 6000 1450

Commit message: C-CAN_Y17 Rev 1.0
This is the C-CAN ordered on march 9th, 2017
Parts:
- added D1: LED, LEDs:LED_0805, symbol LED
- added R8: 1k, Resistors_SMD:R_0805_HandSoldering, symbol R
Connections:
- net +5V: now also R8.1
- net GND: now also D1.1 (K)
- new net: D1.2 (A), R8.2
Changed lines of the file:
@@
 LIBS:switches
 LIBS:C-CAN_Y17-cache
-EELAYER 26 0
+EELAYER 25 0
 EELAYER END
 $Descr A4 11693 8268
@@
 Wire Wire Line
 	4850 6850 5100 6850
+$Comp
+L R R8
+U 1 1 58C2353E
+P 4050 2550
+F 0 "R8" V 4130 2550 50  0000 C CNN
+F 1 "1k" V 4050 2550 50  0000 C CNN
+F 2 "Resistors_SMD:R_0805_HandSoldering" V 3980 2550 50  0001 C CNN
+F 3 "" H 4050 2550 50  0001 C CNN
+	1    4050 2550
+	1    0    0    -1
+$EndComp
+$Comp
+L LED D1
+U 1 1 58C2370D
+P 4050 2950
+F 0 "D1" H 4050 3050 50  0000 C CNN
+F 1 "LED" H 4050 2850 50  0000 C CNN
+F 2 "LEDs:LED_0805" H 4050 2950 50  0001 C CNN
+F 3 "" H 4050 2950 50  0001 C CNN
+	1    4050 2950
+	0    -1   -1   0
+$EndComp
+Wire Wire Line
+	4050 2800 4050 2700
+$Comp
+L +5V #PWR015
+U 1 1 58C2380C
+P 4050 2300
+F 0 "#PWR015" H 4050 2150 50  0001 C CNN
+F 1 "+5V" H 4050 2440 50  0000 C CNN
+F 2 "" H 4050 2300 50  0001 C CNN
+F 3 "" H 4050 2300 50  0001 C CNN
+	1    4050 2300
+	1    0    0    -1
+$EndComp
+Wire Wire Line
+	4050 2300 4050 2400
+$Comp
+L GND #PWR016
+U 1 1 58C238F5
+P 4050 3250
+F 0 "#PWR016" H 4050 3000 50  0001 C CNN
+F 1 "GND" H 4050 3100 50  0000 C CNN
+F 2 "" H 4050 3250 50  0001 C CNN
+F 3 "" H 4050 3250 50  0001 C CNN
+	1    4050 3250
+	1    0    0    -1
+$EndComp
+Wire Wire Line
+	4050 3250 4050 3100
 $EndSCHEMATC
