File: C-CAN_Y17/C-CAN_Y17.kicad_pcb (KiCad board)
At the start: 2 copper layers, 84.5 x 62.2 mm, 19 parts, among them P3 CAN_Terminate, P4 MX150_8, P5 MX150_16, SW1 SW_Push, U1 MCP2551-I/SN, U2 AP1117, U3 Cypress_5LP, Y1 Crystal

Commit message: C-CAN_Y17 Layout done, Oshpark DRC compliant
Still need to do the BOM but everything on the KiCAD side is complete
Parts:
- added J1: S1_Pull, Pin_Headers:Pin_Header_Straight_1x03_Pitch2.54mm, F.Cu at (101.0, 94.0)
- added J2: S2_Pull, Pin_Headers:Pin_Header_Straight_1x03_Pitch2.54mm, F.Cu at (101.0, 102.9)
- added J3: S3_Pull, Pin_Headers:Pin_Header_Straight_1x03_Pitch2.54mm, F.Cu at (105.8, 94.0)
- added J4: S4_Pull, Pin_Headers:Pin_Header_Straight_1x03_Pitch2.54mm, F.Cu at (105.8, 102.9)
- added J5: S5_Pull, Pin_Headers:Pin_Header_Straight_1x03_Pitch2.54mm, F.Cu at (110.7, 94.0)
- added R3: 1M, Resistors_SMD:R_0805_HandSoldering, B.Cu at (98.4, 95.2)
- added R4: 1M, Resistors_SMD:R_0805_HandSoldering, B.Cu at (98.4, 104.1)
- added R5: 1M, Resistors_SMD:R_0805_HandSoldering, B.Cu at (103.4, 95.2)
- added R6: 1M, Resistors_SMD:R_0805_HandSoldering, B.Cu at (103.3, 106.3)
- added R7: 1M, Resistors_SMD:R_0805_HandSoldering, B.Cu at (108.3, 95.1)
Routing:
- net /S4: track 28.4 -> 60.7 mm, vias 0 -> 1
- net /S3: track 48.4 -> 68.2 mm, vias 1 -> 0
- net /S2: track 42.1 -> 52.5 mm, vias 1 -> 2
- net /S1: track 64.5 -> 60.4 mm, vias 0 -> 2
- net Net-(J4-Pad2): track 0.00 -> 3.47 mm
- net Net-(J2-Pad2): track 0.00 -> 2.57 mm
- net Net-(J1-Pad2): track 0.00 -> 2.57 mm
- net Net-(J3-Pad2): track 0.00 -> 2.45 mm
- net Net-(J5-Pad2): track 0.00 -> 2.43 mm
- net /H1: track 39.2 -> 40.9 mm, vias 0 -> 1
Other:
- net class Default: clearance 0.2 -> 0.1524; trace_width 0.25 -> 0.1524; via_dia 0.8 -> 0.6858; via_drill 0.4 -> 0.3302
- rule trace_clearance: 0.2 -> 0.1524
- rule trace_min: 0.2 -> 0.1524
- rule via_min_drill: 0.3 -> 0.3302
- rule via_min_size: 0.4 -> 0.6858

Commit message: Added a bunch of step export files, some solidworks too for the C-CAN_Y17 Enclosure
Parts:
- moved C8 0.25 mm to (130.8, 95.0)
Other:
- board size 84.5 x 62.2 mm -> 84.5 x 57.8 mm
Changed lines of the file:
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@@
     (area 94.9906 66.447599 181.202401 129.259401)
     (thickness 1.6)
-    (drawings 6)
+    (drawings 8)
     (tracks 192)
     (zones 0)
@@
   )
   (module Capacitors_SMD:C_0805_HandSoldering (layer F.Cu)
-    (at 130.81 95.25)
+    (at 130.81 94.996)
     (descr "Capacitor SMD 0805, hand soldering")
     (tags "capacitor 0805")
@@
     )
   )
+  (gr_line (start 96.52 128.905) (end 96.52 128.905) (layer Edge.Cuts) (width 0.15))
+  (gr_line (start 96.52 128.905) (end 96.52 128.905) (layer Edge.Cuts) (width 0.15))
+  (gr_line (start 96.52 71.12) (end 96.52 128.905) (layer Edge.Cuts) (width 0.15))
+  (gr_line (start 180.975 71.12) (end 96.52 71.12) (layer Edge.Cuts) (width 0.15))
+  (gr_line (start 180.975 128.905) (end 180.975 71.12) (layer Edge.Cuts) (width 0.15))
+  (gr_line (start 180.975 128.905) (end 180.975 128.905) (layer Edge.Cuts) (width 0.15))
   (gr_line (start 97.155 66.675) (end 97.155 66.675) (layer Edge.Cuts) (width 0.15))
-  (gr_line (start 96.52 66.675) (end 97.155 66.675) (layer Edge.Cuts) (width 0.15))
-  (gr_line (start 96.52 128.905) (end 96.52 66.675) (layer Edge.Cuts) (width 0.15))
   (gr_line (start 180.975 128.905) (end 96.52 128.905) (layer Edge.Cuts) (width 0.15))
-  (gr_line (start 180.975 66.675) (end 180.975 128.905) (layer Edge.Cuts) (width 0.15))
-  (gr_line (start 97.155 66.675) (end 180.975 66.675) (layer Edge.Cuts) (width 0.15))
   (segment (start 164.465 118.11) (end 161.424001 118.11) (width 0.25) (layer F.Cu) (net 0))
   (segment (start 161.424001 118.11) (end 161.424001 117.691799) (width 0.25) (layer F.Cu) (net 0))
@@
     (polygon
       (pts
-        (xy 180.975 66.675) (xy 96.52 66.675) (xy 96.52 128.905) (xy 180.975 128.905)
+        (xy 180.975 71.12) (xy 96.52 71.12) (xy 96.52 128.905) (xy 180.975 128.905)
       )
     )
@@
       (pts
         (xy 113.03 128.905) (xy 113.03 114.3) (xy 143.51 114.3) (xy 143.51 128.905) (xy 180.975 128.905)
-        (xy 180.975 66.675) (xy 96.52 66.675) (xy 96.52 128.905)
+        (xy 180.975 71.12) (xy 96.52 71.12) (xy 96.52 128.905)
       )
     )

Commit message: C-CAN Fixes
Parts:
- U3: footprint UNCAMotorsports:CypressPSoC -> UNCA Motorsports:PSoC5LP
Connections:
- U1 pad 5: (no net) -> Net-(U1-Pad5)
- U3 pad 12: (no net) -> Net-(U3-Pad12)
- U3 pad 13: (no net) -> Net-(U3-Pad13)
- U3 pad 14: (no net) -> Net-(U3-Pad14)
- U3 pad 15: (no net) -> Net-(U3-Pad15)
- U3 pad 16: (no net) -> Net-(U3-Pad16)
- U3 pad 17: (no net) -> Net-(U3-Pad17)
- U3 pad 18: (no net) -> Net-(U3-Pad18)
- U3 pad 19: (no net) -> Net-(U3-Pad19)
- U3 pad 21: (no net) -> Net-(U3-Pad21)
- U3 pad 22: (no net) -> Net-(U3-Pad22)
- U3 pad 23: (no net) -> Net-(U3-Pad23)
- U3 pad 27: (no net) -> Net-(U3-Pad27)
- U3 pad 28: (no net) -> Net-(U3-Pad28)
- U3 pad 29: (no net) -> Net-(U3-Pad29)
- U3 pad 30: (no net) -> Net-(U3-Pad30)
- U3 pad 31: (no net) -> Net-(U3-Pad31)
- U3 pad 32: (no net) -> Net-(U3-Pad32)
- U3 pad 33: (no net) -> Net-(U3-Pad33)
- U3 pad 34: (no net) -> Net-(U3-Pad34)
- U3 pad 35: (no net) -> Net-(U3-Pad35)
- U3 pad 36: (no net) -> Net-(U3-Pad36)
- U3 pad 37: (no net) -> Net-(U3-Pad37)
- U3 pad 38: (no net) -> Net-(U3-Pad38)
- U3 pad 39: (no net) -> Net-(U3-Pad39)
- U3 pad 4: (no net) -> Net-(U3-Pad4)
- U3 pad 40: (no net) -> Net-(U3-Pad40)
- U3 pad 41: (no net) -> Net-(U3-Pad41)
- U3 pad 42: (no net) -> Net-(U3-Pad42)
- U3 pad 43: (no net) -> Net-(U3-Pad43)
- U3 pad 44: (no net) -> Net-(U3-Pad44)
- U3 pad 45: (no net) -> Net-(U3-Pad45)
- U3 pad 46: (no net) -> Net-(U3-Pad46)
- U3 pad 50: (no net) -> Net-(U3-Pad50)
- U3 pad 7: (no net) -> Net-(U3-Pad7)
- U3 pad 8: (no net) -> Net-(U3-Pad8)
- U3 pad 9: (no net) -> Net-(U3-Pad9)
Routing:
- net /S3: track 68.2 -> 58.1 mm, vias 0 -> 1
- net GND: track 23.4 -> 16.5 mm, vias 5 -> 4
- net /CAN_L: track 69.4 -> 62.7 mm
- net (no net): track 6.17 -> 0.00 mm
- net /H1: track 40.9 -> 37.6 mm
- net Net-(C2-Pad1): track 30.5 -> 27.6 mm
- net Net-(C8-Pad1): track 15.4 -> 17.2 mm
- net Net-(R2-Pad1): track 25.4 -> 23.6 mm
- net +5V: track 14.3 -> 12.6 mm, vias 2 -> 3
- net +12V: track 8.04 -> 6.64 mm, vias 4 -> 0
- net /CAN_H: track 66.9 -> 68.2 mm, vias 1 -> 0
- net /S4: track 60.7 -> 59.5 mm, vias 1 -> 2
- net /S2: track 52.5 -> 51.9 mm, vias 2 -> 0
- net Net-(C7-Pad1): track 11.8 -> 12.3 mm
- net /CAN_TX: track 8.18 -> 8.68 mm
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Other:
- net class Default: trace_width 0.1524 -> 0.254
- net class powah added: clearance 0.1524, trace_width 0.6096, via_dia 0.6858, via_drill 0.3302
- board text added: "UNC Asheville Motorsports Patrick Johnson March 8, 2017"

Commit message: C-CAN_Y17 Rev 1.0
This is the C-CAN ordered on march 9th, 2017
Parts:
- added PWR_GOOD: LED, LEDs:LED_0805, F.Cu at (171.6, 114.8)
- added R8: 1k, Resistors_SMD:R_0805_HandSoldering, F.Cu at (171.6, 119.4)
Connections:
- U1 pad 5: Net-(U1-Pad5) -> (no net)
- U3 pad 12: Net-(U3-Pad12) -> (no net)
- U3 pad 13: Net-(U3-Pad13) -> (no net)
- U3 pad 14: Net-(U3-Pad14) -> (no net)
- U3 pad 15: Net-(U3-Pad15) -> (no net)
- U3 pad 16: Net-(U3-Pad16) -> (no net)
- U3 pad 17: Net-(U3-Pad17) -> (no net)
- U3 pad 18: Net-(U3-Pad18) -> (no net)
- U3 pad 19: Net-(U3-Pad19) -> (no net)
- U3 pad 21: Net-(U3-Pad21) -> (no net)
- U3 pad 22: Net-(U3-Pad22) -> (no net)
- U3 pad 23: Net-(U3-Pad23) -> (no net)
- U3 pad 27: Net-(U3-Pad27) -> (no net)
- U3 pad 28: Net-(U3-Pad28) -> (no net)
- U3 pad 29: Net-(U3-Pad29) -> (no net)
- U3 pad 30: Net-(U3-Pad30) -> (no net)
- U3 pad 31: Net-(U3-Pad31) -> (no net)
- U3 pad 32: Net-(U3-Pad32) -> (no net)
- U3 pad 33: Net-(U3-Pad33) -> (no net)
- U3 pad 34: Net-(U3-Pad34) -> (no net)
- U3 pad 35: Net-(U3-Pad35) -> (no net)
- U3 pad 36: Net-(U3-Pad36) -> (no net)
- U3 pad 37: Net-(U3-Pad37) -> (no net)
- U3 pad 38: Net-(U3-Pad38) -> (no net)
- U3 pad 39: Net-(U3-Pad39) -> (no net)
- U3 pad 4: Net-(U3-Pad4) -> (no net)
- U3 pad 40: Net-(U3-Pad40) -> (no net)
- U3 pad 41: Net-(U3-Pad41) -> (no net)
- U3 pad 42: Net-(U3-Pad42) -> (no net)
- U3 pad 43: Net-(U3-Pad43) -> (no net)
- U3 pad 44: Net-(U3-Pad44) -> (no net)
- U3 pad 45: Net-(U3-Pad45) -> (no net)
- U3 pad 46: Net-(U3-Pad46) -> (no net)
- U3 pad 50: Net-(U3-Pad50) -> (no net)
- U3 pad 7: Net-(U3-Pad7) -> (no net)
- U3 pad 8: Net-(U3-Pad8) -> (no net)
- U3 pad 9: Net-(U3-Pad9) -> (no net)
Routing:
- net Net-(D1-Pad2): track 0.00 -> 2.12 mm
- net GND: track 16.5 -> 18.5 mm, vias 4 -> 5

Commit message: ESF Fixes
Parts:
- removed P4: MX150_8, UNCAMotorsports:MX150_8Pin
- removed P5: MX150_16, UNCAMotorsports:MX150_16pin
- added REF**: MX123_56, UNCAMotorsports:MX123_56, F.Cu at (99.1, 110.5)
- PWR_GOOD, R8: moved to B.Cu
- moved U1 35.0 mm to (137.8, 101.1)
- moved R1 31.1 mm to (137.2, 108.6), turned to 90 degrees
- moved C2 20.7 mm to (143.5, 107.3)
- moved C3 20.7 mm to (147.3, 108.6)
- moved C5 20.7 mm to (144.8, 98.4)
- moved PWR_GOOD 20.7 mm to (157.6, 99.6), turned to 90 degrees
- moved U2 20.7 mm to (149.2, 103.5)
- moved C4 20.7 mm to (143.5, 102.2)
- moved R8 20.7 mm to (157.6, 104.1), turned to 270 degrees
- moved F1 18.8 mm to (150.0, 103.5)
- moved C7 16.5 mm to (118.7, 78.7)
- moved J1 16.5 mm to (101.0, 77.5)
- moved J2 16.5 mm to (101.0, 86.4)
- moved J3 16.5 mm to (105.8, 77.5)
- moved J4 16.5 mm to (105.8, 86.4)
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Routing:
- net /CAN_H: track 68.2 -> 0.00 mm
- net /CAN_L: track 62.7 -> 0.00 mm, vias 1 -> 0
- net /S1: track 60.2 -> 0.00 mm, vias 1 -> 0
- net /S4: track 59.5 -> 0.00 mm, vias 2 -> 0
- net /S3: track 58.1 -> 0.00 mm, vias 1 -> 0
- net /S2: track 51.9 -> 0.00 mm
- net /H1: track 37.6 -> 0.00 mm, vias 1 -> 0
- net Net-(C2-Pad1): track 27.6 -> 0.00 mm, vias 1 -> 0
- net Net-(R2-Pad1): track 23.6 -> 0.00 mm
- net GND: track 18.5 -> 0.00 mm, vias 5 -> 0
- net Net-(C8-Pad1): track 17.2 -> 0.00 mm
- net +5V: track 12.6 -> 0.00 mm, vias 3 -> 0
- net Net-(C7-Pad1): track 12.3 -> 0.00 mm
- net /CAN_TX: track 8.68 -> 0.00 mm
- net /CAN_RX: track 7.66 -> 0.00 mm
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- removed copper zone on F.Cu, net +12V
- removed copper zone on F.Cu, net +5V
Other:
- board size 84.5 x 57.8 mm -> 68.6 x 43.2 mm
