File: VehicleController/file58B1642D.sch (KiCad schematic (older format))
At the start: 10 parts

Commit message: 3D model of 16 pin, MX150_8 pin symbol
Changed lines of the file:
@@
 	6050 3100 5950 3100
 Wire Wire Line
-	6050 2800 6050 2850
-Wire Wire Line
-	6050 2850 6050 3100
+	6050 2800 6050 3100
 $Comp
 L +5VA #PWR?
@@
 $EndComp
 Wire Wire Line
-	6050 2850 6200 2850
-Wire Wire Line
-	6200 2850 6500 2850
+	6050 2850 6500 2850
 Wire Wire Line
 	6200 2850 6200 2900
 Connection ~ 6050 2850
 Wire Wire Line
-	5950 3200 6200 3200
-Wire Wire Line
-	6200 3200 7050 3200
+	5950 3200 7050 3200
 Wire Wire Line
 	6200 3200 6200 3100
@@
 SDA_ISO
 Wire Wire Line
-	5950 3300 6500 3300
-Wire Wire Line
-	6500 3300 7050 3300
+	5950 3300 7050 3300
 Text Label 7050 3300 2    60   ~ 0
 SCL_ISO
@@
 	9350 3250 9700 3250
 Wire Wire Line
-	5800 4550 6000 4550
-Wire Wire Line
-	6000 4550 6750 4550
+	5800 4550 6750 4550
 Text Label 6750 4550 2    60   ~ 0
 LATCH_ISO
@@
 	4900 4750 5200 4750
 Wire Wire Line
-	4200 5100 4500 5100
-Wire Wire Line
-	4500 5100 4600 5100
+	4200 5100 4600 5100
 $Comp
 L GND #PWR?
@@
 $EndComp
 Wire Wire Line
-	4900 5300 4900 5500
-Wire Wire Line
-	4900 5500 4900 5600
+	4900 5300 4900 5600
 $Comp
 L +5V #PWR?

Commit message: Add MX150 8 pin, add Motor Controller connector
Parts:
- added P?: MX150_16, symbol MX150_16
- added RL?: Relay-SPST, symbol Relay-SPST
Connections:
- net labels added: CoilReturn, ContactorL, ContactorR, Fwd, KSI, Mode1, Mode2
- wire segments 49 -> 67
Changed lines of the file:
@@
 LIBS:relays
 LIBS:SystemBlocks
+LIBS:dc-dc
+LIBS:Power_Management
 LIBS:VehicleController-cache
 EELAYER 26 0
@@
 Wire Wire Line
 	4950 2950 4950 3100
+$Comp
+L MX150_16 P?
+U 1 1 58B93178
+P 9650 1800
+F 0 "P?" H 9650 2365 50  0000 C CNN
+F 1 "MX150_16" H 9650 2274 50  0000 C CNN
+F 2 "" H 9650 600 50  0000 C CNN
+F 3 "" H 9650 600 50  0000 C CNN
+	1    9650 1800
+	-1   0    0    -1
+$EndComp
+Wire Wire Line
+	9900 1450 10400 1450
+Text Label 10400 1450 2    60   ~ 0
+KSI
+Text Label 10400 1550 2    60   ~ 0
+Mode1
+Text Label 10400 1650 2    60   ~ 0
+Mode2
+Wire Wire Line
+	10400 1550 9900 1550
+Wire Wire Line
+	9900 1650 10400 1650
+Wire Wire Line
+	10400 1750 9900 1750
+Text Label 10400 1750 2    60   ~ 0
+Fwd
+Wire Wire Line
+	9900 1850 10400 1850
+Text Label 10400 1850 2    60   ~ 0
+ContactorL
+Wire Wire Line
+	9900 2050 10400 2050
+$Comp
+L GNDA #PWR?
+U 1 1 58B932D6
+P 10000 2250
+F 0 "#PWR?" H 10000 2000 50  0001 C CNN
+F 1 "GNDA" H 10005 2077 50  0000 C CNN
+F 2 "" H 10000 2250 50  0000 C CNN
+F 3 "" H 10000 2250 50  0000 C CNN
+	1    10000 2250
+	1    0    0    -1
+$EndComp
+Wire Wire Line
+	9900 2150 10000 2150
+Wire Wire Line
+	10000 2150 10000 2250
+$Comp
+L GNDA #PWR?
+U 1 1 58B93532
+P 9300 2250
+F 0 "#PWR?" H 9300 2000 50  0001 C CNN
+F 1 "GNDA" H 9305 2077 50  0000 C CNN
+F 2 "" H 9300 2250 50  0000 C CNN
+F 3 "" H 9300 2250 50  0000 C CNN
+	1    9300 2250
+	1    0    0    -1
+$EndComp
+Wire Wire Line
+	9300 2250 9300 2150
+Wire Wire Line
+	9300 2150 9400 2150
+Text Label 10400 2050 2    60   ~ 0
+DACL
+Text Label 8850 1450 0    60   ~ 0
+KSI
+Wire Wire Line
+	8850 1450 9400 1450
+Wire Wire Line
+	8850 1550 9400 1550
+Text Label 8850 1550 0    60   ~ 0
+Mode1
+Text Label 8850 1650 0    60   ~ 0
+Mode2
+Text Label 8850 1750 0    60   ~ 0
+Fwd
+Wire Wire Line
+	8850 1750 9400 1750
+Wire Wire Line
+	8850 1650 9400 1650
+Text Label 8850 1850 0    60   ~ 0
+ContactorR
+Wire Wire Line
+	8850 1850 9400 1850
+Wire Wire Line
+	8850 2050 9400 2050
+Text Label 8850 2050 0    60   ~ 0
+DACR
+Wire Wire Line
+	9400 1950 8850 1950
+Text Label 8850 1950 0    60   ~ 0
+CoilReturn
+Wire Wire Line
+	9900 1950 10400 1950
+Text Label 10400 1950 2    60   ~ 0
+CoilReturn
+$Comp
+L Relay-SPST RL?
+U 1 1 58B98C67
+P 8000 1700
+F 0 "RL?" V 7433 1700 50  0000 C CNN
+F 1 "Relay-SPST" V 7524 1700 50  0000 C CNN
+F 2 "" H 8000 1700 50  0000 C CNN
+F 3 "" H 8000 1700 50  0000 C CNN
+	1    8000 1700
+	0    1    1    0
+$EndComp
 $EndSCHEMATC

Commit message: Add High-G Accel, connectors
Parts:
- removed RL?: Relay-SPST, symbol Relay-SPST
- added P7: CONN_01X02, symbol CONN_01X02
- added R12, R14: 4.7k, symbol R_Small
- added U10, U11: Relay_SPST, symbol Relay_SPST
- gave numbers to parts that had none: 11
Connections:
- net labels added: +48V, Shutdown_In, Shutdown_Out
- wire segments 67 -> 90
Other:
- moved on the sheet: Q4, R13, R15, R16, R17, R18, U12, U13, U14, U15

Commit message: Nearly finished with VC Schematic
Parts:
- removed P6: MX150_16, symbol MX150_16
- added P1, P6: MX150_10, symbol MX150_10
- added U17: Relay_SPST, symbol Relay_SPST
Connections:
- net labels added: COILRET, CONTACT_L, CONTACT_R, DAC_L, DAC_R, FWD, ILOCK, MODE1, MODE2, PRECHARGE
- net labels removed: CoilReturn, ContactorL, ContactorR, DACL, DACR, Fwd, Mode1, Mode2
- wire segments 90 -> 98
- no-connect marks 1 -> 3
Other:
- moved on the sheet: P7, Q4, R12, R13, R14, R15, R16, R17, R18, U10, U11, U12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

Commit message: Begin nailing down VC schematic details
Parts:
- removed P7: CONN_01X02, symbol CONN_01X02
- added D11, D12, D13: D, symbol D
- added D14: 5V_ISO, symbol LED_Small_ALT
- added F4: 5A, symbol Fuse
- added J1: CONN_01X03, symbol CONN_01X03
- added Q5: Q_NMOS_GDS, symbol Q_NMOS_GDS
- added R24: 4.7k, symbol R_Small
- added R28: 470, symbol R_Small
- R25: renamed from R15; value 220 -> 470
- U13: renamed from U10; value Relay_SPST -> MCR_Shtdwn
- U14: renamed from U11; value Relay_SPST -> MCL_Shtdwn
- U17: value Relay_SPST -> Precharge
- renumbered P1 to P5, R12 to R21, R13 to R22, R14 to R23, R16 to R26, R17 to R27, R18 to R29, U12 to U15, U13 to U16, U14 to U18, U15 to U19
Connections:
- net +5V: now also Q4.3 (S), R22.2, U17.2, D11.1 (K); no longer R25.2
- net +5VA: now also R28.1
- net DAC_LATCH: now also R22.1; no longer R22.2
- net GND: now also U18.2, Q5.2 (D), R24.2; no longer Q4.3 (S), R22.1, U17.1
- net GNDA: now also D14.1 (K), J1.3 (P3)
- net KSI: now also U13.1, U14.1, F4.2; no longer U17.3
- net PRECHARGE: now also Q5.1 (G), R24.1; no longer U17.2
- net at U18.1: now also R25.2; no longer R25.1
- net at Q4.2 (D): now also R25.1; no longer U18.2
- removed net +48V: U13.1, U14.1, U17.4
- new net: D11.2 (A), Q5.3 (S), U17.1
- new net: D12.1 (K), D13.2 (A), U17.3
- new net: J1.1 (P1), U17.4
- new net: D12.2 (A), J1.2 (P2)
- new net: D13.1 (K), F4.1
- new net: D14.2 (A), R28.2
Other:
- moved on the sheet: P5, P6, R22, R25, U13, U14, U17, U19

Commit message: Finish VCU schematic, most footprint selections.  Start layout
Parts:
- removed J1: CONN_01X03, symbol CONN_01X03
- added J1: MX150_4, UNCAMotorsports:MX150_4, symbol MX150_4
- D11, D12, D13: footprint (none) -> Diodes_SMD:SMA_Handsoldering
- D14: footprint (none) -> LEDs:LED-0805
- P5, P6: footprint (none) -> UNCAMotorsports:MX150_16pin
- Q4, Q5: footprint (none) -> TO_SOT_Packages_SMD:SOT-23_Handsoldering
- R21, R22, R23, R25, R26, R27, R28, R29: footprint (none) -> Resistors_SMD:R_0805_HandSoldering
- R24: value 4.7k -> 10k; footprint (none) -> Resistors_SMD:R_0805_HandSoldering
- U14: renamed from U16; footprint (none) -> SMD_Packages:SOIC-8-N
- U18: footprint DIP-4 -> (none)
- U19: footprint (none) -> Housings_SSOP:TSSOP-8_4.4x3mm_Pitch0.65mm
- renumbered U15 to U13, U17 to U15, U13 to U16, U14 to U17
Connections:
- net labels added: AIR+, TS+
- net labels removed: COILRET
- wire segments 131 -> 116
Other:
- moved on the sheet: P5, P6, U16, U17, U19

Commit message: ESF Fixes
Parts:
- removed F4: 5A, symbol Fuse
- removed J1: MX150_4, UNCAMotorsports:MX150_4, symbol MX150_4
- removed P5, P6: MX150_10, UNCAMotorsports:MX150_16pin, symbol MX150_10
- removed U18: TLP785, symbol TLP785
- added U18: TCMT1103, UNCAMotorsports:SSOP-4, symbol TCMT1103
- added U20: MX123_56, UNCAMotorsports:MX123_56, symbol MX123_56
- Q5: value Q_NMOS_GDS -> PC_FET
- U13: footprint (none) -> UNCAMotorsports:RI-0505S
- U15: value Precharge -> PC_RLY; footprint (none) -> UNCAMotorsports:G6DN-1A
- U16, U17: footprint (none) -> UNCAMotorsports:ALE1PB48
Connections:
- net labels added: FAULT_L1, FAULT_L2, FAULT_R1, FAULT_R2, HV_BATT+, TSMS
- net labels removed: AIR+, FWD, ILOCK, MODE1, MODE2
- wire segments 116 -> 149
- no-connect marks 3 -> 1
