File: VehicleController/file58B1642D.sch (KiCad schematic (older format))
At the start: 41 parts, among them J10 CONN_01X12, J8 CONN_01X03, J9 CONN_01X12, Q4 Q_PMOS_GSD, Q5 Q_NMOS_GSD, Q6 Q_NMOS_GSD, U16 MC_Override, U17 MCR_Shtdwn, U18 MCL_Shtdwn, U19 RI-0505S, U20 ISO1540, U21 TCMT1103, U22 OPTO-TRANSISTOR-4, U23 PC_RLY, U24 MCP47FEBX2

Commit message: Small schematic fixes, start layout
Parts:
- D13, D14, D15, D16, D17, D18: footprint Diodes_SMD:SMC_Handsoldering -> Diodes_SMD:SMA_Handsoldering
- U16: footprint UNCAMotorsports:ALE1PB48 -> UNCAMotorsports:G6DN-1A
Changed lines of the file:
@@
 LIBS:VehicleController-rescue
 LIBS:UNCAMotorsports
-LIBS:power
-LIBS:device
-LIBS:transistors
-LIBS:conn
-LIBS:linear
-LIBS:regul
-LIBS:74xx
-LIBS:cmos4000
-LIBS:adc-dac
-LIBS:memory
-LIBS:xilinx
-LIBS:microcontrollers
-LIBS:dsp
-LIBS:microchip
-LIBS:analog_switches
-LIBS:motorola
-LIBS:texas
-LIBS:intel
-LIBS:audio
-LIBS:interface
-LIBS:digital-audio
-LIBS:philips
-LIBS:display
-LIBS:cypress
-LIBS:siliconi
-LIBS:opto
-LIBS:atmel
-LIBS:contrib
-LIBS:valves
 LIBS:Common-Parts-Library-CPL
 LIBS:relays
 LIBS:SystemBlocks
-LIBS:dc-dc
-LIBS:Power_Management
-LIBS:switches
 LIBS:VehicleController-cache
-EELAYER 25 0
+EELAYER 26 0
 EELAYER END
 $Descr B 17000 11000
@@
 $EndComp
 $Comp
-L +5VA #PWR068
+L +5VA #PWR069
 U 1 1 58B166C2
 P 7850 6250
-F 0 "#PWR068" H 7850 6100 50  0001 C CNN
+F 0 "#PWR069" H 7850 6100 50  0001 C CNN
 F 1 "+5VA" H 7865 6423 50  0000 C CNN
 F 2 "" H 7850 6250 50  0000 C CNN
@@
 $EndComp
 $Comp
-L GNDA #PWR069
+L GNDA #PWR070
 U 1 1 58B166E6
 P 7850 7000
-F 0 "#PWR069" H 7850 6750 50  0001 C CNN
+F 0 "#PWR070" H 7850 6750 50  0001 C CNN
 F 1 "GNDA" H 7855 6827 50  0000 C CNN
 F 2 "" H 7850 7000 50  0000 C CNN
@@
 $EndComp
 $Comp
-L GND #PWR070
+L GND #PWR071
 U 1 1 58B166F7
 P 6750 7000
-F 0 "#PWR070" H 6750 6750 50  0001 C CNN
+F 0 "#PWR071" H 6750 6750 50  0001 C CNN
 F 1 "GND" H 6755 6827 50  0000 C CNN
 F 2 "" H 6750 7000 50  0000 C CNN
@@
 $EndComp
 $Comp
-L +5VA #PWR071
+L +5VA #PWR072
 U 1 1 58B17364
 P 7900 5100
-F 0 "#PWR071" H 7900 4950 50  0001 C CNN
+F 0 "#PWR072" H 7900 4950 50  0001 C CNN
 F 1 "+5VA" H 7915 5273 50  0000 C CNN
 F 2 "" H 7900 5100 50  0000 C CNN
@@
 $EndComp
 $Comp
-L GNDA #PWR072
+L GNDA #PWR073
 U 1 1 58B173AF
 P 7900 5550
-F 0 "#PWR072" H 7900 5300 50  0001 C CNN
+F 0 "#PWR073" H 7900 5300 50  0001 C CNN
 F 1 "GNDA" H 7905 5377 50  0000 C CNN
 F 2 "" H 7900 5550 50  0000 C CNN
@@
 $EndComp
 $Comp
-L GNDA #PWR073
+L GNDA #PWR074
 U 1 1 58B17D44
 P 7700 8200
-F 0 "#PWR073" H 7700 7950 50  0001 C CNN
+F 0 "#PWR074" H 7700 7950 50  0001 C CNN
 F 1 "GNDA" H 7705 8027 50  0000 C CNN
 F 2 "" H 7700 8200 50  0000 C CNN
@@
 NoConn ~ 12500 6000
 $Comp
-L GNDA #PWR074
+L GNDA #PWR075
 U 1 1 58B181A1
 P 10750 6100
-F 0 "#PWR074" H 10750 5850 50  0001 C CNN
+F 0 "#PWR075" H 10750 5850 50  0001 C CNN
 F 1 "GNDA" H 10755 5927 50  0000 C CNN
 F 2 "" H 10750 6100 50  0000 C CNN
@@
 $EndComp
 $Comp
-L +5VA #PWR075
+L +5VA #PWR076
 U 1 1 58B181A7
 P 10750 5500
-F 0 "#PWR075" H 10750 5350 50  0001 C CNN
+F 0 "#PWR076" H 10750 5350 50  0001 C CNN
 F 1 "+5VA" H 10765 5673 50  0000 C CNN
 F 2 "" H 10750 5500 50  0000 C CNN
@@
 $EndComp
 $Comp
-L +5VA #PWR076
+L +5VA #PWR077
 U 1 1 58B1875A
 P 7700 7500
-F 0 "#PWR076" H 7700 7350 50  0001 C CNN
+F 0 "#PWR077" H 7700 7350 50  0001 C CNN
 F 1 "+5VA" H 7715 7673 50  0000 C CNN
 F 2 "" H 7700 7500 50  0000 C CNN
@@
 SCL_IN
 $Comp
-L GND #PWR077
+L GND #PWR078
 U 1 1 58B1731B
 P 6800 5450
-F 0 "#PWR077" H 6800 5200 50  0001 C CNN
+F 0 "#PWR078" H 6800 5200 50  0001 C CNN
 F 1 "GND" H 6805 5277 50  0000 C CNN
 F 2 "" H 6800 5450 50  0000 C CNN
@@
 $EndComp
 $Comp
-L +5V #PWR078
+L +5V #PWR079
 U 1 1 58B172D4
 P 6800 5050
-F 0 "#PWR078" H 6800 4900 50  0001 C CNN
+F 0 "#PWR079" H 6800 4900 50  0001 C CNN
 F 1 "+5V" H 6815 5223 50  0000 C CNN
 F 2 "" H 6800 5050 50  0000 C CNN
@@
 DAC_LATCH
 $Comp
-L +5V #PWR079
+L +5V #PWR080
 U 1 1 58B166EE
 P 6750 6200
-F 0 "#PWR079" H 6750 6050 50  0001 C CNN
+F 0 "#PWR080" H 6750 6050 50  0001 C CNN
 F 1 "+5V" H 6765 6373 50  0000 C CNN
 F 2 "" H 6750 6200 50  0000 C CNN
@@
 CONTACT_R
 $Comp
-L GNDA #PWR080
+L GNDA #PWR081
 U 1 1 58BA1834
 P 11550 4650
-F 0 "#PWR080" H 11550 4400 50  0001 C CNN
+F 0 "#PWR081" H 11550 4400 50  0001 C CNN
 F 1 "GNDA" H 11555 4477 50  0000 C CNN
 F 2 "" H 11550 4650 50  0000 C CNN
@@
 CONTACT_L
 $Comp
-L GNDA #PWR081
+L GNDA #PWR082
 U 1 1 58BA3088
 P 12250 4650
-F 0 "#PWR081" H 12250 4400 50  0001 C CNN
+F 0 "#PWR082" H 12250 4400 50  0001 C CNN
 F 1 "GNDA" H 12255 4477 50  0000 C CNN
 F 2 "" H 12250 4650 50  0000 C CNN
@@
 $EndComp
 $Comp
-L GND #PWR082
+L GND #PWR083
 U 1 1 58BB11C1
 P 7200 2100
-F 0 "#PWR082" H 7200 1850 50  0001 C CNN
+F 0 "#PWR083" H 7200 1850 50  0001 C CNN
 F 1 "GND" H 7205 1927 50  0000 C CNN
 F 2 "" H 7200 2100 50  0000 C CNN
@@
 F 0 "D18" H 8300 1766 50  0000 C CNN
 F 1 "1N4001" H 8300 1675 50  0000 C CNN
-F 2 "Diodes_SMD:SMC_Handsoldering" H -2300 450 50  0001 C CNN
+F 2 "Diodes_SMD:SMA_Handsoldering" H -2300 450 50  0001 C CNN
 F 3 "" H -2300 450 50  0001 C CNN
 	1    8300 1550
@@
 $EndComp
 $Comp
-L GNDA #PWR083
+L GNDA #PWR084
 U 1 1 58C41861
 P 9150 5300
-F 0 "#PWR083" H 9150 5050 50  0001 C CNN
+F 0 "#PWR084" H 9150 5050 50  0001 C CNN
 F 1 "GNDA" H 9155 5127 50  0000 C CNN
 F 2 "" H 9150 5300 50  0000 C CNN
@@
 F 0 "D15" V 7896 1279 50  0000 L CNN
 F 1 "1N4001" V 7805 1279 50  0000 L CNN
-F 2 "Diodes_SMD:SMC_Handsoldering" H -2750 100 50  0001 C CNN
+F 2 "Diodes_SMD:SMA_Handsoldering" H -2750 100 50  0001 C CNN
 F 3 "" H -2750 100 50  0001 C CNN
 	1    7850 1200
@@
 $EndComp
 $Comp
-L GND #PWR084
+L GND #PWR085
 U 1 1 58C501B1
 P 6850 8200
-F 0 "#PWR084" H 6850 7950 50  0001 C CNN
+F 0 "#PWR085" H 6850 7950 50  0001 C CNN
 F 1 "GND" H 6855 8027 50  0000 C CNN
 F 2 "" H 6850 8200 50  0000 C CNN
@@
 F 0 "D14" V 6546 1279 50  0000 L CNN
 F 1 "D" V 6455 1279 50  0000 L CNN
-F 2 "Diodes_SMD:SMC_Handsoldering" H -4100 100 50  0001 C CNN
+F 2 "Diodes_SMD:SMA_Handsoldering" H -4100 100 50  0001 C CNN
 F 3 "" H -4100 100 50  0001 C CNN
 	1    6500 1200
@@
 FAULT_R2
 $Comp
-L GND #PWR085
+L GND #PWR086
 U 1 1 58CAFC96
 P 7700 10150
-F 0 "#PWR085" H 7750 10200 50  0001 C CNN
+F 0 "#PWR086" H 7750 10200 50  0001 C CNN
 F 1 "GND" H 7705 9977 50  0000 C CNN
 F 2 "" H -700 1050 50  0001 C CNN
@@
 F_R2
 $Comp
-L GND #PWR086
+L GND #PWR087
 U 1 1 58CA2742
 P 6900 10150
-F 0 "#PWR086" H 6950 10200 50  0001 C CNN
+F 0 "#PWR087" H 6950 10200 50  0001 C CNN
 F 1 "GND" H 6905 9977 50  0000 C CNN
 F 2 "" H -1500 1050 50  0001 C CNN
@@
 KSI
 $Comp
-L GNDA #PWR087
+L GNDA #PWR088
 U 1 1 590261A6
 P 8400 1050
-F 0 "#PWR087" H 8400 800 50  0001 C CNN
+F 0 "#PWR088" H 8400 800 50  0001 C CNN
 F 1 "GNDA" H 8405 877 50  0000 C CNN
 F 2 "" H 8400 1050 50  0000 C CNN
@@
 F 0 "D17" H 8200 3630 50  0000 L CNN
 F 1 "1N4001" H 8100 3470 50  0000 L CNN
-F 2 "Diodes_SMD:SMC_Handsoldering" V 8250 3550 50  0001 C CNN
+F 2 "Diodes_SMD:SMA_Handsoldering" V 8250 3550 50  0001 C CNN
 F 3 "" V 8250 3550 50  0001 C CNN
 	1    8250 3550
@@
 F 0 "D16" H 8200 3030 50  0000 L CNN
 F 1 "1N4001" H 8100 2870 50  0000 L CNN
-F 2 "Diodes_SMD:SMC_Handsoldering" V 8250 2950 50  0001 C CNN
+F 2 "Diodes_SMD:SMA_Handsoldering" V 8250 2950 50  0001 C CNN
 F 3 "" V 8250 2950 50  0001 C CNN
 	1    8250 2950
@@
 $EndComp
 $Comp
-L +5V #PWR088
+L +5V #PWR089
 U 1 1 59116008
 P 5500 6500
-F 0 "#PWR088" H 5500 6350 50  0001 C CNN
+F 0 "#PWR089" H 5500 6350 50  0001 C CNN
 F 1 "+5V" H 5515 6673 50  0000 C CNN
 F 2 "" H 5500 6500 50  0000 C CNN
@@
 $EndComp
 $Comp
-L GND #PWR089
+L GND #PWR090
 U 1 1 5911608E
 P 5500 6900
-F 0 "#PWR089" H 5500 6650 50  0001 C CNN
+F 0 "#PWR090" H 5500 6650 50  0001 C CNN
 F 1 "GND" H 5505 6727 50  0000 C CNN
 F 2 "" H 5500 6900 50  0000 C CNN
@@
 $EndComp
 $Comp
-L +5VA #PWR090
+L +5VA #PWR091
 U 1 1 591164A6
 P 9100 6500
-F 0 "#PWR090" H 9100 6350 50  0001 C CNN
+F 0 "#PWR091" H 9100 6350 50  0001 C CNN
 F 1 "+5VA" H 9115 6673 50  0000 C CNN
 F 2 "" H 9100 6500 50  0000 C CNN
@@
 	9100 6500 9100 6600
 $Comp
-L GNDA #PWR091
+L GNDA #PWR092
 U 1 1 5911666B
 P 9100 6900
-F 0 "#PWR091" H 9100 6650 50  0001 C CNN
+F 0 "#PWR092" H 9100 6650 50  0001 C CNN
 F 1 "GNDA" H 9105 6727 50  0000 C CNN
 F 2 "" H 9100 6900 50  0000 C CNN
@@
 F 0 "U16" V 6747 3528 60  0000 L CNN
 F 1 "MC_Override" V 6853 3528 60  0000 L CNN
-F 2 "UNCAMotorsports:ALE1PB48" H 6800 3250 60  0001 C CNN
+F 2 "UNCAMotorsports:G6DN-1A" H 6800 3250 60  0001 C CNN
 F 3 "" H 6800 3250 60  0001 C CNN
 	1    6800 3250
@@
 	6650 3450 6650 3600
 $Comp
-L GND #PWR092
+L GND #PWR093
 U 1 1 591496EE
 P 6650 4150
-F 0 "#PWR092" H 6650 3900 50  0001 C CNN
+F 0 "#PWR093" H 6650 3900 50  0001 C CNN
 F 1 "GND" H 6655 3977 50  0000 C CNN
 F 2 "" H 6650 4150 50  0000 C CNN
@@
 Connection ~ 6250 3800
 $Comp
-L +5V #PWR093
+L +5V #PWR094
 U 1 1 5914B610
 P 6650 2950
-F 0 "#PWR093" H 6650 2800 50  0001 C CNN
+F 0 "#PWR094" H 6650 2800 50  0001 C CNN
 F 1 "+5V" H 6650 3090 50  0000 C CNN
 F 2 "" H 6650 2950 50  0001 C CNN
@@
 F 0 "D13" V 5896 3329 50  0000 L CNN
 F 1 "D" V 5805 3329 50  0000 L CNN
-F 2 "Diodes_SMD:SMC_Handsoldering" H -4750 2150 50  0001 C CNN
+F 2 "Diodes_SMD:SMA_Handsoldering" H -4750 2150 50  0001 C CNN
 F 3 "" H -4750 2150 50  0001 C CNN
 	1    5850 3250

Commit message: Major layout of VCU begins.  Moved some nets to facilitate layout
Parts:
- added TP1, TP2, TP3, TP4: TEST, Measurement_Points:Measurement_Point_Round-SMD-Pad_Big, symbol TEST
Connections:
- net +5V: now also TP1.1
- net GND: now also TP2.1
- net GNDA: now also TP4.1
- net KSI: now also TP3.1
Changed lines of the file:
@@
 LIBS:VehicleController-rescue
 LIBS:UNCAMotorsports
+LIBS:power
+LIBS:device
+LIBS:transistors
+LIBS:conn
+LIBS:linear
+LIBS:regul
+LIBS:74xx
+LIBS:cmos4000
+LIBS:adc-dac
+LIBS:memory
+LIBS:xilinx
+LIBS:microcontrollers
+LIBS:dsp
+LIBS:microchip
+LIBS:analog_switches
+LIBS:motorola
+LIBS:texas
+LIBS:intel
+LIBS:audio
+LIBS:interface
+LIBS:digital-audio
+LIBS:philips
+LIBS:display
+LIBS:cypress
+LIBS:siliconi
+LIBS:opto
+LIBS:atmel
+LIBS:contrib
+LIBS:valves
 LIBS:Common-Parts-Library-CPL
 LIBS:relays
 LIBS:SystemBlocks
+LIBS:dc-dc
+LIBS:Power_Management
+LIBS:switches
 LIBS:VehicleController-cache
-EELAYER 26 0
+EELAYER 25 0
 EELAYER END
 $Descr B 17000 11000
@@
 	1    0    0    -1
 $EndComp
+$Comp
+L TEST TP1
+U 1 1 59267245
+P 3250 1350
+F 0 "TP1" H 3250 1650 50  0000 C BNN
+F 1 "TEST" H 3250 1600 50  0000 C CNN
+F 2 "Measurement_Points:Measurement_Point_Round-SMD-Pad_Big" H 3250 1350 50  0001 C CNN
+F 3 "" H 3250 1350 50  0001 C CNN
+	1    3250 1350
+	0    1    1    0
+$EndComp
+$Comp
+L TEST TP2
+U 1 1 592677FE
+P 3250 1550
+F 0 "TP2" H 3250 1850 50  0000 C BNN
+F 1 "TEST" H 3250 1800 50  0000 C CNN
+F 2 "Measurement_Points:Measurement_Point_Round-SMD-Pad_Big" H 3250 1550 50  0001 C CNN
+F 3 "" H 3250 1550 50  0001 C CNN
+	1    3250 1550
+	0    1    1    0
+$EndComp
+$Comp
+L TEST TP3
+U 1 1 592678A8
+P 10250 750
+F 0 "TP3" H 10250 1050 50  0000 C BNN
+F 1 "TEST" H 10250 1000 50  0000 C CNN
+F 2 "Measurement_Points:Measurement_Point_Round-SMD-Pad_Big" H 10250 750 50  0001 C CNN
+F 3 "" H 10250 750 50  0001 C CNN
+	1    10250 750
+	0    -1   -1   0
+$EndComp
+$Comp
+L TEST TP4
+U 1 1 59267E34
+P 10250 1000
+F 0 "TP4" H 10250 1300 50  0000 C BNN
+F 1 "TEST" H 10250 1250 50  0000 C CNN
+F 2 "Measurement_Points:Measurement_Point_Round-SMD-Pad_Big" H 10250 1000 50  0001 C CNN
+F 3 "" H 10250 1000 50  0001 C CNN
+	1    10250 1000
+	0    -1   -1   0
+$EndComp
+$Comp
+L GNDA #PWR095
+U 1 1 59267FA8
+P 10350 1100
+F 0 "#PWR095" H 10350 850 50  0001 C CNN
+F 1 "GNDA" H 10355 927 50  0000 C CNN
+F 2 "" H 10350 1100 50  0000 C CNN
+F 3 "" H 10350 1100 50  0000 C CNN
+	1    10350 1100
+	1    0    0    -1
+$EndComp
+Wire Wire Line
+	10250 1000 10350 1000
+Wire Wire Line
+	10350 1000 10350 1100
+$Comp
+L +5V #PWR096
+U 1 1 59269684
+P 3150 1250
+F 0 "#PWR096" H 3150 1100 50  0001 C CNN
+F 1 "+5V" H 3150 1390 50  0000 C CNN
+F 2 "" H 3150 1250 50  0001 C CNN
+F 3 "" H 3150 1250 50  0001 C CNN
+	1    3150 1250
+	1    0    0    -1
+$EndComp
+Wire Wire Line
+	3150 1250 3150 1350
+Wire Wire Line
+	3150 1350 3250 1350
+$Comp
+L GND #PWR097
+U 1 1 59269CB2
+P 3150 1700
+F 0 "#PWR097" H 3150 1450 50  0001 C CNN
+F 1 "GND" H 3155 1527 50  0000 C CNN
+F 2 "" H 3150 1700 50  0000 C CNN
+F 3 "" H 3150 1700 50  0000 C CNN
+	1    3150 1700
+	1    0    0    -1
+$EndComp
+Wire Wire Line
+	3150 1700 3150 1550
+Wire Wire Line
+	3150 1550 3250 1550
+Text Label 10500 750  2    60   ~ 0
+KSI
+Wire Wire Line
+	10250 750  10500 750
 $EndSCHEMATC

Commit message: VCU layout progress
Connections:
- net GND: no longer U22.2, U22.4, U22.6, U22.8
- net GNDA: now also U22.2, U22.4, U22.6, U22.8
Changed lines of the file:
@@
 Text Label 8400 9850 2    60   ~ 0
 FAULT_R2
-$Comp
-L GND #PWR086
-U 1 1 58CAFC96
-P 7700 10150
-F 0 "#PWR086" H 7750 10200 50  0001 C CNN
-F 1 "GND" H 7705 9977 50  0000 C CNN
-F 2 "" H -700 1050 50  0001 C CNN
-F 3 "" H -700 1050 50  0001 C CNN
-	1    7700 10150
-	1    0    0    -1
-$EndComp
 Text HLabel 6750 8650 0    60   Input ~ 0
 F_L1
@@
 Wire Wire Line
 	10250 750  10500 750
+$Comp
+L GNDA #PWR?
+U 1 1 5926F8B7
+P 7700 10150
+F 0 "#PWR?" H 7700 9900 50  0001 C CNN
+F 1 "GNDA" H 7700 10000 50  0000 C CNN
+F 2 "" H 7700 10150 50  0001 C CNN
+F 3 "" H 7700 10150 50  0001 C CNN
+	1    7700 10150
+	1    0    0    -1
+$EndComp
 $EndSCHEMATC
