File: VehicleController/file58B2371B.sch (KiCad schematic (older format))
At the start: 7 parts

Commit message: Added GPS, DAC, Isolation sheet, buzzer to VC
Parts:
- added C?: C_Small, symbol C_Small
Connections:
- net GND: now also C?.2
- net VBACKUP: now also C?.1
Changed lines of the file:
@@
 $Descr A4 11693 8268
 encoding utf-8
-Sheet 3 4
+Sheet 3 5
 Title ""
 Date ""
@@
 	1    0    0    -1
 $EndComp
-Text HLabel 6250 3150 0    60   Input ~ 0
+Text HLabel 6050 3150 0    60   Input ~ 0
 3D-FIX
 Text HLabel 6250 3550 0    60   Input ~ 0
@@
 Text HLabel 6250 3650 0    60   Input ~ 0
 GPS_RX
-Text HLabel 6250 3050 0    60   Input ~ 0
+Text HLabel 6050 3050 0    60   Input ~ 0
 VBACKUP
 $Comp
@@
 Connection ~ 8100 3550
 Wire Wire Line
-	6250 3150 6500 3150
+	6050 3150 6500 3150
 Wire Wire Line
 	6250 3550 6500 3550
@@
 Connection ~ 6400 3450
 Wire Wire Line
-	6250 3050 6500 3050
+	6050 3050 6500 3050
 Wire Wire Line
 	4000 3300 4250 3300
@@
 Connection ~ 6150 2850
 NoConn ~ 7500 3350
+$Comp
+L C_Small C?
+U 1 1 58B346B2
+P 6250 3300
+F 0 "C?" H 6342 3346 50  0000 L CNN
+F 1 "C_Small" H 6342 3255 50  0000 L CNN
+F 2 "" H 6250 3300 50  0000 C CNN
+F 3 "" H 6250 3300 50  0000 C CNN
+	1    6250 3300
+	-1   0    0    -1
+$EndComp
+Wire Wire Line
+	6250 3200 6250 3050
+Connection ~ 6250 3050
+Wire Wire Line
+	6250 3400 6250 3450
+Connection ~ 6250 3450
 $EndSCHEMATC

Commit message: Add High-G Accel, connectors
Parts:
- gave numbers to parts that had none: 8
Changed lines of the file:
@@
 LIBS:dc-dc
 LIBS:Power_Management
+LIBS:switches
 LIBS:VehicleController-cache
 EELAYER 26 0
@@
 $EndDescr
 $Comp
-L FGMMOPA6H U?
+L FGMMOPA6H U7
 U 1 1 58B2411D
 P 6950 3150
-F 0 "U?" H 7000 3837 60  0000 C CNN
+F 0 "U7" H 7000 3837 60  0000 C CNN
 F 1 "FGMMOPA6H" H 7000 3731 60  0000 C CNN
 F 2 "" H 6950 3400 60  0000 C CNN
@@
 $EndComp
 $Comp
-L C_Small C?
+L C_Small C9
 U 1 1 58B24124
 P 5450 3000
-F 0 "C?" H 5542 3046 50  0000 L CNN
+F 0 "C9" H 5542 3046 50  0000 L CNN
 F 1 "C_Small" H 5542 2955 50  0000 L CNN
 F 2 "" H 5450 3000 50  0000 C CNN
@@
 $EndComp
 $Comp
-L R_Small R?
+L R_Small R10
 U 1 1 58B2412B
 P 6150 2600
-F 0 "R?" V 6250 2600 50  0000 C CNN
+F 0 "R10" V 6250 2600 50  0000 C CNN
 F 1 "10k" V 6050 2600 50  0000 C CNN
 F 2 "" H 6150 2600 50  0000 C CNN
@@
 $EndComp
 $Comp
-L GND #PWR?
+L GND #PWR33
 U 1 1 58B24137
 P 5450 3800
-F 0 "#PWR?" H 5450 3550 50  0001 C CNN
+F 0 "#PWR33" H 5450 3550 50  0001 C CNN
 F 1 "GND" H 5455 3627 50  0000 C CNN
 F 2 "" H 5450 3800 50  0000 C CNN
@@
 $EndComp
 $Comp
-L U.FL_Antenna U?
+L U.FL_Antenna U8
 U 1 1 58B24140
 P 7850 3650
-F 0 "U?" H 7700 3500 60  0000 C CNN
+F 0 "U8" H 7700 3500 60  0000 C CNN
 F 1 "U.FL_Antenna" H 8150 3800 60  0001 C CNN
 F 2 "" H 7850 3650 60  0000 C CNN
@@
 $EndComp
 $Comp
-L GND #PWR?
+L GND #PWR34
 U 1 1 58B24148
 P 8100 4050
-F 0 "#PWR?" H 8100 3800 50  0001 C CNN
+F 0 "#PWR34" H 8100 3800 50  0001 C CNN
 F 1 "GND" H 8105 3877 50  0000 C CNN
 F 2 "" H 8100 4050 50  0000 C CNN
@@
 VBACKUP
 $Comp
-L +3.3V #PWR?
+L +3.3V #PWR32
 U 1 1 58B276E4
 P 5450 2300
-F 0 "#PWR?" H 5450 2150 50  0001 C CNN
+F 0 "#PWR32" H 5450 2150 50  0001 C CNN
 F 1 "+3.3V" H 5465 2473 50  0000 C CNN
 F 2 "" H 5450 2300 50  0000 C CNN
@@
 $EndComp
 $Comp
-L GND #PWR?
+L GND #PWR31
 U 1 1 58B23C84
 P 3700 3600
-F 0 "#PWR?" H 3700 3350 50  0001 C CNN
+F 0 "#PWR31" H 3700 3350 50  0001 C CNN
 F 1 "GND" H 3705 3427 50  0000 C CNN
 F 2 "" H 3700 3600 50  0000 C CNN
@@
 $EndComp
 $Comp
-L Q_NMOS_GDS Q?
+L Q_NMOS_GDS Q3
 U 1 1 58B23C7C
 P 3800 3300
-F 0 "Q?" H 4006 3346 50  0000 L CNN
+F 0 "Q3" H 4006 3346 50  0000 L CNN
 F 1 "Q_NMOS_GDS" H 4006 3255 50  0000 L CNN
 F 2 "" H 4000 3400 50  0000 C CNN
@@
 $EndComp
 $Comp
-L +3.3V #PWR?
+L +3.3V #PWR30
 U 1 1 58B23C75
 P 3700 2400
-F 0 "#PWR?" H 3700 2250 50  0001 C CNN
+F 0 "#PWR30" H 3700 2250 50  0001 C CNN
 F 1 "+3.3V" H 3715 2573 50  0000 C CNN
 F 2 "" H 3700 2400 50  0000 C CNN
@@
 $EndComp
 $Comp
-L R_Small R?
+L R_Small R9
 U 1 1 58B23C6D
 P 3700 2600
-F 0 "R?" H 3759 2646 50  0000 L CNN
+F 0 "R9" H 3759 2646 50  0000 L CNN
 F 1 "R_Small" H 3759 2555 50  0000 L CNN
 F 2 "" H 3700 2600 50  0000 C CNN
@@
 $EndComp
 $Comp
-L LED_Small D?
+L LED_Small D3
 U 1 1 58B23C66
 P 3700 2900
-F 0 "D?" V 3746 2832 50  0000 R CNN
+F 0 "D3" V 3746 2832 50  0000 R CNN
 F 1 "LED_Small" V 3655 2832 50  0000 R CNN
 F 2 "" V 3700 2900 50  0000 C CNN
@@
 NoConn ~ 7500 3350
 $Comp
-L C_Small C?
+L C_Small C10
 U 1 1 58B346B2
 P 6250 3300
-F 0 "C?" H 6342 3346 50  0000 L CNN
+F 0 "C10" H 6342 3346 50  0000 L CNN
 F 1 "C_Small" H 6342 3255 50  0000 L CNN
 F 2 "" H 6250 3300 50  0000 C CNN

Commit message: Begin nailing down VC schematic details
Parts:
- removed D3: LED_Small, symbol LED_Small
- added D8: 3DFix, symbol LED_Small_ALT
- C10: renamed from C9; value C_Small -> 0.1uF
- C11: renamed from C10; value C_Small -> 0.1uF
- R16: renamed from R9; value R_Small -> 220
- renumbered R10 to R17, U8 to U10, U7 to U9
Connections:
- net at Q3.2 (D): now also D8.1 (K)
- net at R16.2: now also D8.2 (A)
Changed lines of the file:
@@
 $EndDescr
 $Comp
-L FGMMOPA6H U7
+L FGMMOPA6H U9
 U 1 1 58B2411D
 P 6950 3150
-F 0 "U7" H 7000 3837 60  0000 C CNN
+F 0 "U9" H 7000 3837 60  0000 C CNN
 F 1 "FGMMOPA6H" H 7000 3731 60  0000 C CNN
 F 2 "" H 6950 3400 60  0000 C CNN
@@
 $EndComp
 $Comp
-L C_Small C9
+L C_Small C10
 U 1 1 58B24124
 P 5450 3000
-F 0 "C9" H 5542 3046 50  0000 L CNN
-F 1 "C_Small" H 5542 2955 50  0000 L CNN
+F 0 "C10" H 5542 3046 50  0000 L CNN
+F 1 "0.1uF" H 5542 2955 50  0000 L CNN
 F 2 "" H 5450 3000 50  0000 C CNN
 F 3 "" H 5450 3000 50  0000 C CNN
@@
 $EndComp
 $Comp
-L R_Small R10
+L R_Small R17
 U 1 1 58B2412B
 P 6150 2600
-F 0 "R10" V 6250 2600 50  0000 C CNN
+F 0 "R17" V 6250 2600 50  0000 C CNN
 F 1 "10k" V 6050 2600 50  0000 C CNN
 F 2 "" H 6150 2600 50  0000 C CNN
@@
 $EndComp
 $Comp
-L GND #PWR035
+L GND #PWR39
 U 1 1 58B24137
 P 5450 3800
-F 0 "#PWR035" H 5450 3550 50  0001 C CNN
+F 0 "#PWR39" H 5450 3550 50  0001 C CNN
 F 1 "GND" H 5455 3627 50  0000 C CNN
 F 2 "" H 5450 3800 50  0000 C CNN
@@
 $EndComp
 $Comp
-L U.FL_Antenna U8
+L U.FL_Antenna U10
 U 1 1 58B24140
 P 7850 3650
-F 0 "U8" H 7700 3500 60  0000 C CNN
+F 0 "U10" H 7700 3500 60  0000 C CNN
 F 1 "U.FL_Antenna" H 8150 3800 60  0001 C CNN
 F 2 "" H 7850 3650 60  0000 C CNN
@@
 $EndComp
 $Comp
-L GND #PWR036
+L GND #PWR40
 U 1 1 58B24148
 P 8100 4050
-F 0 "#PWR036" H 8100 3800 50  0001 C CNN
+F 0 "#PWR40" H 8100 3800 50  0001 C CNN
 F 1 "GND" H 8105 3877 50  0000 C CNN
 F 2 "" H 8100 4050 50  0000 C CNN
@@
 VBACKUP
 $Comp
-L +3.3V #PWR037
+L +3.3V #PWR38
 U 1 1 58B276E4
 P 5450 2300
-F 0 "#PWR037" H 5450 2150 50  0001 C CNN
+F 0 "#PWR38" H 5450 2150 50  0001 C CNN
 F 1 "+3.3V" H 5465 2473 50  0000 C CNN
 F 2 "" H 5450 2300 50  0000 C CNN
@@
 $EndComp
 $Comp
-L GND #PWR038
+L GND #PWR37
 U 1 1 58B23C84
 P 3700 3600
-F 0 "#PWR038" H 3700 3350 50  0001 C CNN
+F 0 "#PWR37" H 3700 3350 50  0001 C CNN
 F 1 "GND" H 3705 3427 50  0000 C CNN
 F 2 "" H 3700 3600 50  0000 C CNN
@@
 $EndComp
 $Comp
-L +3.3V #PWR039
+L +3.3V #PWR36
 U 1 1 58B23C75
 P 3700 2400
-F 0 "#PWR039" H 3700 2250 50  0001 C CNN
+F 0 "#PWR36" H 3700 2250 50  0001 C CNN
 F 1 "+3.3V" H 3715 2573 50  0000 C CNN
 F 2 "" H 3700 2400 50  0000 C CNN
@@
 $EndComp
 $Comp
-L R_Small R9
+L R_Small R16
 U 1 1 58B23C6D
 P 3700 2600
-F 0 "R9" H 3759 2646 50  0000 L CNN
-F 1 "R_Small" H 3759 2555 50  0000 L CNN
+F 0 "R16" H 3759 2646 50  0000 L CNN
+F 1 "220" H 3759 2555 50  0000 L CNN
 F 2 "" H 3700 2600 50  0000 C CNN
 F 3 "" H 3700 2600 50  0000 C CNN
 	1    3700 2600
 	1    0    0    -1
-$EndComp
-$Comp
-L LED_Small D3
-U 1 1 58B23C66
-P 3700 2900
-F 0 "D3" V 3746 2832 50  0000 R CNN
-F 1 "LED_Small" V 3655 2832 50  0000 R CNN
-F 2 "" V 3700 2900 50  0000 C CNN
-F 3 "" V 3700 2900 50  0000 C CNN
-	1    3700 2900
-	0    -1   -1   0
 $EndComp
 Text HLabel 4250 3300 2    60   Input ~ 0
@@
 NoConn ~ 7500 3350
 $Comp
-L C_Small C10
+L C_Small C11
 U 1 1 58B346B2
 P 6250 3300
-F 0 "C10" H 6342 3346 50  0000 L CNN
-F 1 "C_Small" H 6342 3255 50  0000 L CNN
+F 0 "C11" H 6342 3346 50  0000 L CNN
+F 1 "0.1uF" H 6342 3255 50  0000 L CNN
 F 2 "" H 6250 3300 50  0000 C CNN
 F 3 "" H 6250 3300 50  0000 C CNN
@@
 	6250 3400 6250 3450
 Connection ~ 6250 3450
+$Comp
+L LED_Small_ALT D8
+U 1 1 58C36B03
+P 3700 2900
+F 0 "D8" V 3746 2832 50  0000 R CNN
+F 1 "3DFix" V 3655 2832 50  0000 R CNN
+F 2 "" V 0   0   50  0001 C CNN
+F 3 "" V 0   0   50  0001 C CNN
+	1    3700 2900
+	0    -1   -1   0
+$EndComp
 $EndSCHEMATC

Commit message: Finish VCU schematic, most footprint selections.  Start layout
Parts:
- C10, C11: footprint (none) -> Capacitors_SMD:C_0805_HandSoldering
- D8: footprint (none) -> LEDs:LED-0805
- Q3: footprint (none) -> TO_SOT_Packages_SMD:SOT-23_Handsoldering
- R16, R17: footprint (none) -> Resistors_SMD:R_0805_HandSoldering
- U10: footprint (none) -> UNCAMotorsports:U.FL-CON
- U9: footprint (none) -> UNCAMotorsports:GPS_16x16
Changed lines of the file:
@@
 encoding utf-8
 Sheet 3 5
-Title ""
-Date ""
-Rev ""
-Comp ""
+Title "Vehicle Controller"
+Date "2017-03-11"
+Rev "001"
+Comp "UNC Asheville Motorsports"
 Comment1 ""
 Comment2 ""
@@
 F 0 "U9" H 7000 3837 60  0000 C CNN
 F 1 "FGMMOPA6H" H 7000 3731 60  0000 C CNN
-F 2 "" H 6950 3400 60  0000 C CNN
+F 2 "UNCAMotorsports:GPS_16x16" H 6950 3400 60  0001 C CNN
 F 3 "" H 6950 3400 60  0000 C CNN
 	1    6950 3150
@@
 F 0 "C10" H 5542 3046 50  0000 L CNN
 F 1 "0.1uF" H 5542 2955 50  0000 L CNN
-F 2 "" H 5450 3000 50  0000 C CNN
+F 2 "Capacitors_SMD:C_0805_HandSoldering" H 5450 3000 50  0001 C CNN
 F 3 "" H 5450 3000 50  0000 C CNN
 	1    5450 3000
@@
 F 0 "R17" V 6250 2600 50  0000 C CNN
 F 1 "10k" V 6050 2600 50  0000 C CNN
-F 2 "" H 6150 2600 50  0000 C CNN
+F 2 "Resistors_SMD:R_0805_HandSoldering" H 6150 2600 50  0001 C CNN
 F 3 "" H 6150 2600 50  0000 C CNN
 	1    6150 2600
@@
 $EndComp
 $Comp
-L GND #PWR39
+L GND #PWR039
 U 1 1 58B24137
 P 5450 3800
-F 0 "#PWR39" H 5450 3550 50  0001 C CNN
+F 0 "#PWR039" H 5450 3550 50  0001 C CNN
 F 1 "GND" H 5455 3627 50  0000 C CNN
 F 2 "" H 5450 3800 50  0000 C CNN
@@
 F 0 "U10" H 7700 3500 60  0000 C CNN
 F 1 "U.FL_Antenna" H 8150 3800 60  0001 C CNN
-F 2 "" H 7850 3650 60  0000 C CNN
+F 2 "UNCAMotorsports:U.FL-CON" H 7850 3650 60  0001 C CNN
 F 3 "" H 7850 3650 60  0000 C CNN
 	1    7850 3650
@@
 $EndComp
 $Comp
-L GND #PWR40
+L GND #PWR040
 U 1 1 58B24148
 P 8100 4050
-F 0 "#PWR40" H 8100 3800 50  0001 C CNN
+F 0 "#PWR040" H 8100 3800 50  0001 C CNN
 F 1 "GND" H 8105 3877 50  0000 C CNN
 F 2 "" H 8100 4050 50  0000 C CNN
@@
 VBACKUP
 $Comp
-L +3.3V #PWR38
+L +3.3V #PWR041
 U 1 1 58B276E4
 P 5450 2300
-F 0 "#PWR38" H 5450 2150 50  0001 C CNN
+F 0 "#PWR041" H 5450 2150 50  0001 C CNN
 F 1 "+3.3V" H 5465 2473 50  0000 C CNN
 F 2 "" H 5450 2300 50  0000 C CNN
@@
 $EndComp
 $Comp
-L GND #PWR37
+L GND #PWR042
 U 1 1 58B23C84
 P 3700 3600
-F 0 "#PWR37" H 3700 3350 50  0001 C CNN
+F 0 "#PWR042" H 3700 3350 50  0001 C CNN
 F 1 "GND" H 3705 3427 50  0000 C CNN
 F 2 "" H 3700 3600 50  0000 C CNN
@@
 F 0 "Q3" H 4006 3346 50  0000 L CNN
 F 1 "Q_NMOS_GDS" H 4006 3255 50  0000 L CNN
-F 2 "" H 4000 3400 50  0000 C CNN
+F 2 "TO_SOT_Packages_SMD:SOT-23_Handsoldering" H 4000 3400 50  0001 C CNN
 F 3 "" H 3800 3300 50  0000 C CNN
 	1    3800 3300
@@
 $EndComp
 $Comp
-L +3.3V #PWR36
+L +3.3V #PWR043
 U 1 1 58B23C75
 P 3700 2400
-F 0 "#PWR36" H 3700 2250 50  0001 C CNN
+F 0 "#PWR043" H 3700 2250 50  0001 C CNN
 F 1 "+3.3V" H 3715 2573 50  0000 C CNN
 F 2 "" H 3700 2400 50  0000 C CNN
@@
 F 0 "R16" H 3759 2646 50  0000 L CNN
 F 1 "220" H 3759 2555 50  0000 L CNN
-F 2 "" H 3700 2600 50  0000 C CNN
+F 2 "Resistors_SMD:R_0805_HandSoldering" H 3700 2600 50  0001 C CNN
 F 3 "" H 3700 2600 50  0000 C CNN
 	1    3700 2600
@@
 F 0 "C11" H 6342 3346 50  0000 L CNN
 F 1 "0.1uF" H 6342 3255 50  0000 L CNN
-F 2 "" H 6250 3300 50  0000 C CNN
+F 2 "Capacitors_SMD:C_0805_HandSoldering" H 6250 3300 50  0001 C CNN
 F 3 "" H 6250 3300 50  0000 C CNN
 	1    6250 3300
@@
 F 0 "D8" V 3746 2832 50  0000 R CNN
 F 1 "3DFix" V 3655 2832 50  0000 R CNN
-F 2 "" V 0   0   50  0001 C CNN
+F 2 "LEDs:LED-0805" V 0   0   50  0001 C CNN
 F 3 "" V 0   0   50  0001 C CNN
 	1    3700 2900
