File: VehicleController/PowerDistribution.sch (KiCad schematic (older format))
At the start: 21 parts, among them P2 RPi_USB_PWR, U6 TL431, U7 BTS6133D, U8 R-78E5.0-1.0

Commit message: ESF Fixes
Parts:
- U8: footprint (none) -> UNCAMotorsports:R-78Cxx-1.0
Changed lines of the file:
@@
 LIBS:switches
 LIBS:VehicleController-cache
-EELAYER 26 0
+EELAYER 25 0
 EELAYER END
 $Descr A4 11693 8268
@@
 $EndComp
 $Comp
-L GND #PWR028
+L GND #PWR030
 U 1 1 587C7BE3
 P 6000 3550
-F 0 "#PWR028" H 6000 3300 50  0001 C CNN
+F 0 "#PWR030" H 6000 3300 50  0001 C CNN
 F 1 "GND" H 6005 3377 50  0000 C CNN
 F 2 "" H 6000 3550 50  0000 C CNN
@@
 $EndComp
 $Comp
-L GND #PWR029
+L GND #PWR031
 U 1 1 587C7BF7
 P 4300 4700
-F 0 "#PWR029" H 4300 4450 50  0001 C CNN
+F 0 "#PWR031" H 4300 4450 50  0001 C CNN
 F 1 "GND" H 4305 4527 50  0000 C CNN
 F 2 "" H 4300 4700 50  0000 C CNN
@@
 $EndComp
 $Comp
-L GND #PWR030
+L GND #PWR032
 U 1 1 58AEB860
 P 8650 3250
-F 0 "#PWR030" H 8650 3000 50  0001 C CNN
+F 0 "#PWR032" H 8650 3000 50  0001 C CNN
 F 1 "GND" H 8655 3077 50  0000 C CNN
 F 2 "" H 8650 3250 50  0000 C CNN
@@
 5V
 $Comp
-L PWR_FLAG #FLG031
+L PWR_FLAG #FLG033
 U 1 1 58AF2028
 P 5550 1000
-F 0 "#FLG031" H 5550 1095 50  0001 C CNN
+F 0 "#FLG033" H 5550 1095 50  0001 C CNN
 F 1 "PWR_FLAG" H 5550 1224 50  0001 C CNN
 F 2 "" H 5550 1000 50  0000 C CNN
@@
 $EndComp
 $Comp
-L GND #PWR032
+L GND #PWR034
 U 1 1 58B30D9F
 P 8900 5300
-F 0 "#PWR032" H 8900 5050 50  0001 C CNN
+F 0 "#PWR034" H 8900 5050 50  0001 C CNN
 F 1 "GND" H 8905 5127 50  0000 C CNN
 F 2 "" H 8900 5300 50  0000 C CNN
@@
 12V
 $Comp
-L GND #PWR033
+L GND #PWR035
 U 1 1 58B31164
 P 9650 5100
-F 0 "#PWR033" H 9650 4850 50  0001 C CNN
+F 0 "#PWR035" H 9650 4850 50  0001 C CNN
 F 1 "GND" H 9655 4927 50  0000 C CNN
 F 2 "" H 9650 5100 50  0000 C CNN
@@
 $EndComp
 $Comp
-L GND #PWR034
+L GND #PWR036
 U 1 1 58B0EFE3
 P 3350 3250
-F 0 "#PWR034" H 3350 3000 50  0001 C CNN
+F 0 "#PWR036" H 3350 3000 50  0001 C CNN
 F 1 "GND" H 3355 3077 50  0000 C CNN
 F 2 "" H 3350 3250 50  0000 C CNN
@@
 $EndComp
 $Comp
-L GND #PWR035
+L GND #PWR037
 U 1 1 58B0F09D
 P 3550 3250
-F 0 "#PWR035" H 3550 3000 50  0001 C CNN
+F 0 "#PWR037" H 3550 3000 50  0001 C CNN
 F 1 "GND" H 3555 3077 50  0000 C CNN
 F 2 "" H 3550 3250 50  0000 C CNN
@@
 	4850 3300 4850 3550
 $Comp
-L +5V #PWR036
+L +5V #PWR038
 U 1 1 58BE7A1A
 P 9300 2600
-F 0 "#PWR036" H 9350 2650 50  0001 C CNN
+F 0 "#PWR038" H 9350 2650 50  0001 C CNN
 F 1 "+5V" H 9315 2773 50  0000 C CNN
 F 2 "" H 550 -100 50  0001 C CNN
@@
 Connection ~ 7500 2750
 $Comp
-L GND #PWR037
+L GND #PWR039
 U 1 1 58C31B60
 P 7500 3500
-F 0 "#PWR037" H 7500 3250 50  0001 C CNN
+F 0 "#PWR039" H 7500 3250 50  0001 C CNN
 F 1 "GND" H 7505 3327 50  0000 C CNN
 F 2 "" H 7500 3500 50  0000 C CNN
@@
 	9650 3200 9650 3150
 $Comp
-L GND #PWR038
+L GND #PWR040
 U 1 1 58C32364
 P 9650 3500
-F 0 "#PWR038" H 9650 3250 50  0001 C CNN
+F 0 "#PWR040" H 9650 3250 50  0001 C CNN
 F 1 "GND" H 9655 3327 50  0000 C CNN
 F 2 "" H 9650 3500 50  0000 C CNN
@@
 F 0 "U8" H 8650 3037 60  0000 C CNN
 F 1 "R-78E5.0-1.0" H 8650 2931 60  0000 C CNN
-F 2 "" H 2600 1150 60  0001 C CNN
+F 2 "UNCAMotorsports:R-78Cxx-1.0" H 2600 1150 60  0001 C CNN
 F 3 "" H 2600 1150 60  0000 C CNN
 	1    8650 2750

Commit message: More updates prior to finalizing design
Parts:
- added D17: 3.3V, symbol D_Zener_Small
- R27: renamed from R13; value 1k -> 620
- renumbered D4 to D6, D5 to D7, D6 to D8, D7 to D9, F3 to F10, F2 to F9, P2 to P3, R10 to R24, R11 to R25, R12 to R26, R14 to R28, R15 to R29, U7 to U10, U8 to U11, U6 to U9
Connections:
- net CurrentSense: now also D17.1 (K)
- net GND: now also D17.2 (A)
Other:
- moved on the sheet: R27
Changed lines of the file:
@@
 $EndDescr
 $Comp
-L D_Schottky D4
+L D_Schottky D6
 U 1 1 587C7BB2
 P 3000 2750
-F 0 "D4" H 3000 2534 50  0000 C CNN
+F 0 "D6" H 3000 2534 50  0000 C CNN
 F 1 "D_Schottky" H 3000 2625 50  0000 C CNN
 F 2 "Diodes_SMD:SMA_Handsoldering" H 3000 2750 50  0001 C CNN
@@
 $EndComp
 $Comp
-L Polyfuse F2
+L Polyfuse F9
 U 1 1 587C7BB9
 P 2450 2750
-F 0 "F2" V 2225 2750 50  0000 C CNN
+F 0 "F9" V 2225 2750 50  0000 C CNN
 F 1 "10A" V 2316 2750 50  0000 C CNN
 F 2 "" H 2500 2550 50  0001 L CNN
@@
 $EndComp
 $Comp
-L TL431 U6
+L TL431 U9
 U 1 1 587C7BC0
 P 4850 3850
-F 0 "U6" H 4671 3903 60  0000 R CNN
+F 0 "U9" H 4671 3903 60  0000 R CNN
 F 1 "TL431" H 4671 3797 60  0000 R CNN
 F 2 "TO_SOT_Packages_SMD:SOT-23_Handsoldering" H 4850 3800 60  0001 C CNN
@@
 $EndComp
 $Comp
-L BTS6133D U7
+L BTS6133D U10
 U 1 1 587C7BC7
 P 6550 2850
-F 0 "U7" H 6550 3237 60  0000 C CNN
+F 0 "U10" H 6550 3237 60  0000 C CNN
 F 1 "BTS6133D" H 6550 3131 60  0000 C CNN
 F 2 "UNCAMotorsports:TO-252-5" H 6700 3050 60  0001 C CNN
@@
 $EndComp
 $Comp
-L R R10
+L R R24
 U 1 1 587C7BCE
 P 4300 3550
-F 0 "R10" H 4369 3596 50  0000 L CNN
+F 0 "R24" H 4369 3596 50  0000 L CNN
 F 1 "330k" H 4369 3505 50  0000 L CNN
 F 2 "Resistors_SMD:R_0805_HandSoldering" V 4230 3550 50  0001 C CNN
@@
 $EndComp
 $Comp
-L R R11
+L R R25
 U 1 1 587C7BD5
 P 4300 4100
-F 0 "R11" H 4369 4146 50  0000 L CNN
+F 0 "R25" H 4369 4146 50  0000 L CNN
 F 1 "120k" H 4369 4055 50  0000 L CNN
 F 2 "Resistors_SMD:R_0805_HandSoldering" V 4230 4100 50  0001 C CNN
@@
 $EndComp
 $Comp
-L R R13
+L R R27
 U 1 1 587C7BDC
-P 6000 3300
-F 0 "R13" H 6069 3346 50  0000 L CNN
-F 1 "1k" H 6069 3255 50  0000 L CNN
-F 2 "Resistors_SMD:R_0805_HandSoldering" V 5930 3300 50  0001 C CNN
-F 3 "" H 6000 3300 50  0000 C CNN
-	1    6000 3300
-	-1   0    0    -1
-$EndComp
-$Comp
-L GND #PWR36
+P 5850 3300
+F 0 "R27" H 5919 3346 50  0000 L CNN
+F 1 "620" H 5919 3255 50  0000 L CNN
+F 2 "Resistors_SMD:R_0805_HandSoldering" V 5780 3300 50  0001 C CNN
+F 3 "" H 5850 3300 50  0000 C CNN
+	1    5850 3300
+	-1   0    0    -1
+$EndComp
+$Comp
+L GND #PWR040
 U 1 1 587C7BE3
-P 6000 3550
-F 0 "#PWR36" H 6000 3300 50  0001 C CNN
-F 1 "GND" H 6005 3377 50  0000 C CNN
-F 2 "" H 6000 3550 50  0000 C CNN
-F 3 "" H 6000 3550 50  0000 C CNN
-	1    6000 3550
-	1    0    0    -1
-$EndComp
-$Comp
-L GND #PWR35
+P 5850 3650
+F 0 "#PWR040" H 5850 3400 50  0001 C CNN
+F 1 "GND" H 5855 3477 50  0000 C CNN
+F 2 "" H 5850 3650 50  0000 C CNN
+F 3 "" H 5850 3650 50  0000 C CNN
+	1    5850 3650
+	1    0    0    -1
+$EndComp
+$Comp
+L GND #PWR041
 U 1 1 587C7BF7
 P 4300 4700
-F 0 "#PWR35" H 4300 4450 50  0001 C CNN
+F 0 "#PWR041" H 4300 4450 50  0001 C CNN
 F 1 "GND" H 4305 4527 50  0000 C CNN
 F 2 "" H 4300 4700 50  0000 C CNN
@@
 Text HLabel 2000 2750 0    60   Input ~ 0
 PWR_IN
-Text HLabel 5800 2950 0    60   Input ~ 0
+Text HLabel 5650 2950 0    60   Input ~ 0
 CurrentSense
 $Comp
@@
 $EndComp
 $Comp
-L GND #PWR38
+L GND #PWR042
 U 1 1 58AEB860
 P 8650 3250
-F 0 "#PWR38" H 8650 3000 50  0001 C CNN
+F 0 "#PWR042" H 8650 3000 50  0001 C CNN
 F 1 "GND" H 8655 3077 50  0000 C CNN
 F 2 "" H 8650 3250 50  0000 C CNN
@@
 5V
 $Comp
-L PWR_FLAG #FLG3
+L PWR_FLAG #FLG043
 U 1 1 58AF2028
 P 5550 1000
-F 0 "#FLG3" H 5550 1095 50  0001 C CNN
+F 0 "#FLG043" H 5550 1095 50  0001 C CNN
 F 1 "PWR_FLAG" H 5550 1224 50  0001 C CNN
 F 2 "" H 5550 1000 50  0000 C CNN
@@
 12V
 $Comp
-L USB_A-RESCUE-VehicleController P2
+L USB_A-RESCUE-VehicleController P3
 U 1 1 58B30D8B
 P 9000 4900
-F 0 "P2" V 8575 4824 50  0000 C CNN
+F 0 "P3" V 8575 4824 50  0000 C CNN
 F 1 "RPi_USB_PWR" V 8666 4824 50  0000 C CNN
 F 2 "UNCAMotorsports:USB-A-THT" V 8950 4800 50  0001 C CNN
@@
 $EndComp
 $Comp
-L GND #PWR39
+L GND #PWR044
 U 1 1 58B30D9F
 P 8900 5300
-F 0 "#PWR39" H 8900 5050 50  0001 C CNN
+F 0 "#PWR044" H 8900 5050 50  0001 C CNN
 F 1 "GND" H 8905 5127 50  0000 C CNN
 F 2 "" H 8900 5300 50  0000 C CNN
@@
 12V
 $Comp
-L GND #PWR42
+L GND #PWR045
 U 1 1 58B31164
 P 9650 5100
-F 0 "#PWR42" H 9650 4850 50  0001 C CNN
+F 0 "#PWR045" H 9650 4850 50  0001 C CNN
 F 1 "GND" H 9655 4927 50  0000 C CNN
 F 2 "" H 9650 5100 50  0000 C CNN
@@
 $EndComp
 $Comp
-L GND #PWR33
+L GND #PWR046
 U 1 1 58B0EFE3
 P 3350 3250
-F 0 "#PWR33" H 3350 3000 50  0001 C CNN
+F 0 "#PWR046" H 3350 3000 50  0001 C CNN
 F 1 "GND" H 3355 3077 50  0000 C CNN
 F 2 "" H 3350 3250 50  0000 C CNN
@@
 $EndComp
 $Comp
-L GND #PWR34
+L GND #PWR047
 U 1 1 58B0F09D
 P 3550 3250
-F 0 "#PWR34" H 3550 3000 50  0001 C CNN
+F 0 "#PWR047" H 3550 3000 50  0001 C CNN
 F 1 "GND" H 3555 3077 50  0000 C CNN
 F 2 "" H 3550 3250 50  0000 C CNN
@@
 $EndComp
 $Comp
-L D_ALT D5
+L D_ALT D7
 U 1 1 58B90308
 P 5400 3850
-F 0 "D5" V 5354 3929 50  0000 L CNN
+F 0 "D7" V 5354 3929 50  0000 L CNN
 F 1 "D_ALT" V 5445 3929 50  0000 L CNN
 F 2 "Diodes_SMD:SMA_Handsoldering" H 5400 3850 50  0001 C CNN
@@
 $EndComp
 Wire Wire Line
-	6000 3150 6000 2950
-Wire Wire Line
-	5800 2950 6150 2950
+	5850 3150 5850 2950
+Wire Wire Line
+	5650 2950 6150 2950
 Wire Wire Line
 	4850 2850 6150 2850
@@
 Connection ~ 4300 2750
 Wire Wire Line
-	6000 3550 6000 3450
+	5850 3450 5850 3650
 Wire Wire Line
 	4300 3700 4300 3950
@@
 	7150 2850 7150 2750
 Connection ~ 7150 2750
-Connection ~ 6000 2950
+Connection ~ 5850 2950
 Wire Wire Line
 	8650 3050 8650 3250
@@
 	4850 3300 4850 3550
 $Comp
-L +5V #PWR40
+L +5V #PWR048
 U 1 1 58BE7A1A
 P 9300 2600
-F 0 "#PWR40" H 9350 2650 50  0001 C CNN
+F 0 "#PWR048" H 9350 2650 50  0001 C CNN
 F 1 "+5V" H 9315 2773 50  0000 C CNN
 F 2 "" H 550 -100 50  0001 C CNN
@@
 Connection ~ 9300 2750
 $Comp
-L Polyfuse F3
+L Polyfuse F10
 U 1 1 58C2ADFE
 P 7850 2750
-F 0 "F3" V 7625 2750 50  0000 C CNN
+F 0 "F10" V 7625 2750 50  0000 C CNN
 F 1 "1A" V 7716 2750 50  0000 C CNN
 F 2 "Fuse_Holders_and_Fuses:Fuse_SMD1206_HandSoldering" H 7900 2550 50  0001 L CNN
@@
 $EndComp
 $Comp
-L R R14
+L R R28
 U 1 1 58C314B1
 P 7500 3000
-F 0 "R14" H 7569 3046 50  0000 L CNN
+F 0 "R28" H 7569 3046 50  0000 L CNN
 F 1 "2.2k" H 7569 2955 50  0000 L CNN
 F 2 "Resistors_SMD:R_0805_HandSoldering" V 7430 3000 50  0001 C CNN
@@
 $EndComp
 $Comp
-L LED_Small_ALT D6
+L LED_Small_ALT D8
 U 1 1 58C318C7
 P 7500 3300
-F 0 "D6" V 7546 3232 50  0000 R CNN
+F 0 "D8" V 7546 3232 50  0000 R CNN
 F 1 "12V_Status" V 7455 3232 50  0000 R CNN
 F 2 "LEDs:LED-0805" V 750 -300 50  0001 C CNN
@@
 Connection ~ 7500 2750
 $Comp
-L GND #PWR37
+L GND #PWR049
 U 1 1 58C31B60
 P 7500 3500
-F 0 "#PWR37" H 7500 3250 50  0001 C CNN
+F 0 "#PWR049" H 7500 3250 50  0001 C CNN
 F 1 "GND" H 7505 3327 50  0000 C CNN
 F 2 "" H 7500 3500 50  0000 C CNN
@@
 	7500 3500 7500 3400
 $Comp
-L LED_Small_ALT D7
+L LED_Small_ALT D9
 U 1 1 58C3218B
 P 9650 3300
-F 0 "D7" V 9696 3232 50  0000 R CNN
+F 0 "D9" V 9696 3232 50  0000 R CNN
 F 1 "5V_Status" V 9605 3232 50  0000 R CNN
 F 2 "LEDs:LED-0805" V 2900 -300 50  0001 C CNN
@@
 $EndComp
 $Comp
-L R R15
+L R R29
 U 1 1 58C321FD
 P 9650 3000
-F 0 "R15" H 9719 3046 50  0000 L CNN
+F 0 "R29" H 9719 3046 50  0000 L CNN
 F 1 "470" H 9719 2955 50  0000 L CNN
 F 2 "Resistors_SMD:R_0805_HandSoldering" V 9580 3000 50  0001 C CNN
@@
 	9650 3200 9650 3150
 $Comp
-L GND #PWR41
+L GND #PWR050
 U 1 1 58C32364
 P 9650 3500
-F 0 "#PWR41" H 9650 3250 50  0001 C CNN
+F 0 "#PWR050" H 9650 3250 50  0001 C CNN
 F 1 "GND" H 9655 3327 50  0000 C CNN
 F 2 "" H 9650 3500 50  0000 C CNN
@@
 $EndComp
 $Comp
-L R R12
+L R R26
 U 1 1 58C342F9
 P 4850 3150
-F 0 "R12" H 4919 3196 50  0000 L CNN
+F 0 "R26" H 4919 3196 50  0000 L CNN
 F 1 "0R" H 4919 3105 50  0000 L CNN
 F 2 "Resistors_SMD:R_0805_HandSoldering" V 4780 3150 50  0001 C CNN
@@
 	4850 3000 4850 2850
 $Comp
-L R-78E5.0-1.0 U8
+L R-78E5.0-1.0 U11
 U 1 1 58C571BC
 P 8650 2750
-F 0 "U8" H 8650 3037 60  0000 C CNN
+F 0 "U11" H 8650 3037 60  0000 C CNN
 F 1 "R-78E5.0-1.0" H 8650 2931 60  0000 C CNN
 F 2 "UNCAMotorsports:R-78Cxx-1.0" H 2600 1150 60  0001 C CNN
@@
 	1    0    0    -1
 $EndComp
+Connection ~ 5850 3550
+$Comp
+L D_Zener_Small D17
+U 1 1 58FBF2F0
+P 6050 3300
+F 0 "D17" H 6050 3390 50  0000 C CNN
+F 1 "3.3V" H 6050 3210 50  0000 C CNN
+F 2 "" V 6050 3300 50  0001 C CNN
+F 3 "" V 6050 3300 50  0001 C CNN
+	1    6050 3300
+	0    1    1    0
+$EndComp
+Wire Wire Line
+	6050 3200 6050 2950
+Connection ~ 6050 2950
+Wire Wire Line
+	6050 3400 6050 3550
+Wire Wire Line
+	6050 3550 5850 3550
 $EndSCHEMATC
