File: VehicleController/PowerDistribution.sch (KiCad schematic (older format))
At the start: 27 parts, among them J11 RPI_PWR, U10 BTS6133D, U11 R-78E5.0-1.0, U25 V7805W-2000, U9 TL431

Commit message: VCU Finalization, BOM generation
Parts:
- C18: value 22u -> 22uF
- C9: value 10u -> 10uF
Changed lines of the file:
@@
 P 7250 4400
 F 0 "C9" H 7275 4500 50  0000 L CNN
-F 1 "10u" H 7275 4300 50  0000 L CNN
+F 1 "10uF" H 7275 4300 50  0000 L CNN
 F 2 "Capacitors_SMD:C_0805_HandSoldering" H 7288 4250 50  0001 C CNN
 F 3 "" H 7250 4400 50  0001 C CNN
@@
 P 8200 4400
 F 0 "C18" H 8225 4500 50  0000 L CNN
-F 1 "22u" H 8225 4300 50  0000 L CNN
+F 1 "22uF" H 8225 4300 50  0000 L CNN
 F 2 "Capacitors_SMD:C_0805_HandSoldering" H 8238 4250 50  0001 C CNN
 F 3 "" H 8200 4400 50  0001 C CNN
