File: VehicleController/VehicleController.kicad_pcb (KiCad board)
At the start: 2 copper layers, 3.4 x 3.4 mm, 81 parts, among them J1 MX150_4, P1 MX150_8, P2 RPi_USB_PWR, P3 CONN_01X02, P4 MX150_8, P5 MX150_10, P6 MX150_10, Q1 Q_NMOS_GDS, Q2 Q_PMOS_GDS, Q3 Q_NMOS_GDS, Q4 Q_NMOS_GDS, Q5 Q_NMOS_GDS, U1 BTS6133D, U10 U.FL_Antenna, U11 NDC7002N, U12 MCP2551, U14 ISO1540, U19 MCP47FEBX2, U2 H3LIS331DL, U4 Teensy_3.5, U5 NDC7003P, U6 TL431, U7 BTS6133D, U9 FGMMOPA6H

Commit message: ESF Fixes
Parts:
- removed J1: MX150_4, UNCAMotorsports:MX150_4
- removed P5, P6: MX150_10, UNCAMotorsports:MX150_16pin
- added U13: RI-0505S, UNCAMotorsports:RI-0505S, F.Cu at (142.2, 48.3)
- added U15: Precharge, UNCAMotorsports:G6DN-1A, F.Cu at (56.5, 62.2)
- added U16: MCR_Shtdwn, UNCAMotorsports:ALE1PB48, F.Cu at (17.8, 44.5)
- added U17: MCL_Shtdwn, UNCAMotorsports:ALE1PB48, F.Cu at (33.0, 44.5)
- added U18: TCMT1103, UNCAMotorsports:SSOP-4, F.Cu at (154.9, 47.0)
- added U20: MX123_56, UNCAMotorsports:MX123_56, F.Cu at (19.1, 31.9)
- added U3: UltimateSensorFusion, UNCAMotorsports:UltimateSensorFusion, F.Cu at (47.0, 85.1)
- added U8: R-78E5.0-1.0, UNCAMotorsports:R-78Cxx-1.0, F.Cu at (176.3, 64.8)
- Q1: value Q_NMOS_GDS -> Shutdown_FET
- moved C11 206.4 mm to (41.9, 121.9)
- moved C10 200.6 mm to (47.0, 121.9), turned to 180 degrees
- moved D8 197.7 mm to (50.8, 134.6), turned to 270 degrees
- moved R17 195.4 mm to (47.0, 124.5)
- moved Q3 192.2 mm to (49.9, 129.5)
- moved R16 189.3 mm to (50.8, 139.7), turned to 90 degrees
- moved U10 189.1 mm to (32.4, 146.9), turned to 180 degrees
- moved C6 165.9 mm to (215.3, 46.2)
- moved U7 140.0 mm to (191.3, 45.8), turned to 0 degrees
- moved U9 133.4 mm to (39.1, 135.0), turned to 270 degrees
- moved C5 126.1 mm to (187.2, 62.1), turned to 0 degrees
- moved P4 108.0 mm to (44.9, 173.7), turned to 0 degrees
- moved D14 86.2 mm to (145.8, 43.2)
- moved R13 84.7 mm to (221.9, 51.4)
- moved R14 84.5 mm to (221.5, 45.1)
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Connections:
- D12 pad 2: /Isolation/TS+ -> (no net)
- P1 pad 3: (no net) -> /SHTDWN_OUT
- P2 pad SHD: (no net) -> GND
- R25 pad 2: (no net) -> Net-(R25-Pad2)
- U2 pad 11: (no net) -> Net-(U2-Pad11)
- U2 pad 4: (no net) -> Net-(U2-Pad4)
- U2 pad 6: (no net) -> Net-(U2-Pad6)
- U2 pad 9: (no net) -> /HighG
- U4 pad 39: (no net) -> /IMU_INT
Routing:
- added copper zone on F.Cu, net /Isolation/KSI
- added copper zone on B.Cu, net GND
- added copper zone on B.Cu, net GNDA
Other:
- net class Default: clearance 0.2032 -> 0.2; trace_width 0.254 -> 0.25
- rule pad_to_mask_clearance: 0.2 -> 0
- rule trace_clearance: 0.2032 -> 0.2

Commit message: Re-do MX120, GDS->GSD, Associations.
Parts:
- removed C1: 10uF_Al, Capacitors_SMD:c_elec_5x5.8
- removed C10, C11: 0.1uF, Capacitors_SMD:C_0805_HandSoldering
- removed C12, C3, C4: 1uF, Capacitors_SMD:C_0805_HandSoldering
- removed C2: 100nF, Capacitors_SMD:C_0805_HandSoldering
- removed C5: 100uF_Al, Capacitors_SMD:c_elec_6.3x7.7
- removed C6: 1uF_Al, Capacitors_SMD:c_elec_4x4.5
- removed C7, C8: 10uF, Capacitors_SMD:C_0805_HandSoldering
- removed C9: 1uF_Al, Capacitors_SMD:c_elec_4x5.3
- removed D1: 3.1v, Diodes_SMD:SMA_Handsoldering
- removed D10: CANRX, LEDs:LED-0805
- removed D11, D12, D13: D, Diodes_SMD:SMA_Handsoldering
- removed D14: 5V_ISO, LEDs:LED-0805
- removed D2: SCL0, LEDs:LED-0805
- removed D3: SDA0, LEDs:LED-0805
- removed D4: D_Schottky, Diodes_SMD:SMA_Handsoldering
- removed D5: D_ALT, Diodes_SMD:SMA_Handsoldering
- removed D6: 12V_Status, LEDs:LED-0805
- removed D7: 5V_Status, LEDs:LED-0805
- removed D8: 3DFix, LEDs:LED-0805
- removed D9: CANTX, LEDs:LED-0805
- removed F1, F3: 1A, Fuse_Holders_and_Fuses:Fuse_SMD1206_HandSoldering
- removed P1, P4: MX150_8, UNCAMotorsports:MX150_8Pin
- removed P2: RPi_USB_PWR, UNCAMotorsports:USB-A-THT
- removed P3: CONN_01X02, Pin_Headers:Pin_Header_Angled_1x02
- removed Q1: Shutdown_FET, TO_SOT_Packages_SMD:SOT-23_Handsoldering
- removed Q2: Q_PMOS_GDS, TO_SOT_Packages_SMD:SOT-23_Handsoldering
- removed Q3, Q4, Q5: Q_NMOS_GDS, TO_SOT_Packages_SMD:SOT-23_Handsoldering
- removed R1, R17, R22, R24, R26, R4, R5, R7: 10k, Resistors_SMD:R_0805_HandSoldering
- removed R10: 330k, Resistors_SMD:R_0805_HandSoldering
- removed R11: 120k, Resistors_SMD:R_0805_HandSoldering
- removed R12, R2: 0R, Resistors_SMD:R_0805_HandSoldering
- removed R13, R3: 1k, Resistors_SMD:R_0805_HandSoldering
- removed R14, R6: 2.2k, Resistors_SMD:R_0805_HandSoldering
- removed R15, R25, R28: 470, Resistors_SMD:R_0805_HandSoldering
- removed R16, R19, R20, R8, R9: 220, Resistors_SMD:R_0805_HandSoldering
- removed R18: 120, Resistors_SMD:R_0805_HandSoldering
- removed R21, R23, R27, R29: 4.7k, Resistors_SMD:R_0805_HandSoldering
- removed U1, U7: BTS6133D, UNCAMotorsports:TO-252-5
- removed U10: U.FL_Antenna, UNCAMotorsports:U.FL-CON
- removed U11: NDC7002N, TO_SOT_Packages_SMD:SOT-23-6
- removed U12: MCP2551, SMD_Packages:SOIC-8-N
- removed U13: RI-0505S, UNCAMotorsports:RI-0505S
- removed U14: ISO1540, SMD_Packages:SOIC-8-N
- removed U15: Precharge, UNCAMotorsports:G6DN-1A
- removed U16: MCR_Shtdwn, UNCAMotorsports:ALE1PB48
- removed U17: MCL_Shtdwn, UNCAMotorsports:ALE1PB48
- removed U18: TCMT1103, UNCAMotorsports:SSOP-4
- removed U19: MCP47FEBX2, Housings_SSOP:TSSOP-8_4.4x3mm_Pitch0.65mm
- removed U2: H3LIS331DL, UNCAMotorsports:LGA-16-3x3
- removed U20: MX123_56, UNCAMotorsports:MX123_56
- removed U3: UltimateSensorFusion, UNCAMotorsports:UltimateSensorFusion
- removed U4: Teensy_3.5, UNCAMotorsports:Teensy_3.5
- removed U5: NDC7003P, TO_SOT_Packages_SMD:SOT-23-6
- removed U6: TL431, TO_SOT_Packages_SMD:SOT-23_Handsoldering
- removed U8: R-78E5.0-1.0, UNCAMotorsports:R-78Cxx-1.0
- removed U9: FGMMOPA6H, UNCAMotorsports:GPS_16x16
Routing:
- removed copper zone on F.Cu, net /Isolation/KSI
- removed copper zone on B.Cu, net GND
- removed copper zone on B.Cu, net GNDA
Other:
- board outline removed
- net class Default: via_dia 0.8 -> 0.6

Commit message: Library Fixes
Parts:
- added BT1: CR1220, UNCAMotorsports:BATT_CR1220, F.Cu at (148.5, 105.0)
- added C1: 10uF_Al, Capacitors_SMD:c_elec_5x5.8, F.Cu at (148.5, 105.0)
- added C10, C11: 0.1uF, Capacitors_SMD:C_0805_HandSoldering, F.Cu at (148.5, 105.0)
- added C12, C13, C16, C17, C3, C4: 1uF, Capacitors_SMD:C_0805_HandSoldering, F.Cu at (148.5, 105.0)
- added C14, C15, C7, C8: 10uF, Capacitors_SMD:C_0805_HandSoldering, F.Cu at (148.5, 105.0)
- added C2: 100nF, Capacitors_SMD:C_0805_HandSoldering, F.Cu at (148.5, 105.0)
- added C5: 100uF_Al, Capacitors_SMD:c_elec_6.3x7.7, F.Cu at (148.5, 105.0)
- added C6: 1uF_Al, Capacitors_SMD:C_0805_HandSoldering, F.Cu at (148.5, 105.0)
- added D1, D2, D7: 3.3V, Diodes_SMD:SOD-323, F.Cu at (148.5, 105.0)
- added D10: 3DFix, LEDs:LED-0805, F.Cu at (148.5, 105.0)
- added D11: CANTX, LEDs:LED-0805, F.Cu at (148.5, 105.0)
- added D12: CANRX, LEDs:LED-0805, F.Cu at (148.5, 105.0)
- added D13, D14: D, Diodes_SMD:SMC_Handsoldering, F.Cu at (148.5, 105.0)
- added D15, D16, D17, D18: 1N4001, Diodes_SMD:SMC_Handsoldering, F.Cu at (148.5, 105.0)
- added D19: 5V_ISO, LEDs:LED-0805, F.Cu at (148.5, 105.0)
- added D3: SCL0, LEDs:LED-0805, F.Cu at (148.5, 105.0)
- added D4: SDA0, LEDs:LED-0805, F.Cu at (148.5, 105.0)
- added D5: D_Schottky, Diodes_SMD:SMC_Handsoldering, F.Cu at (148.5, 105.0)
- added D6: D_ALT, Diodes_SMD:SMC_Handsoldering, F.Cu at (148.5, 105.0)
- added D8: 12V_Status, LEDs:LED-0805, F.Cu at (148.5, 105.0)
- added D9: 5V_Status, LEDs:LED-0805, F.Cu at (148.5, 105.0)
- added F1, F2, F3, F4, F5, F6, F7, F8, F9: 3A, Resistors_SMD:R_1210_HandSoldering, F.Cu at (148.5, 105.0)
- added F10: 1A, Resistors_SMD:R_1210_HandSoldering, F.Cu at (148.5, 105.0)
- added J1: CONN_02X06, UNCAMotorsports:MX120G-12, F.Cu at (148.5, 105.0)
- added J10, J9: CONN_01X12, UNCAMotorsports:MX120G-12, F.Cu at (148.5, 105.0)
- added J2: USF_SLAVE_I2C, Pin_Headers:Pin_Header_Straight_1x03, F.Cu at (148.5, 105.0)
- added J5: I2C_0, Pin_Headers:Pin_Header_Straight_1x03, F.Cu at (148.5, 105.0)
- added J6: I2C_1, Pin_Headers:Pin_Header_Straight_1x03, F.Cu at (148.5, 105.0)
- added J7: CAN_SER, Pin_Headers:Pin_Header_Straight_1x03, F.Cu at (148.5, 105.0)
- added J8: CONN_01X03, Pin_Headers:Pin_Header_Straight_1x03, F.Cu at (148.5, 105.0)
- added P1, P2: OUTPUTS, UNCAMotorsports:MX120G-12, F.Cu at (148.5, 105.0)
- added P4: CONN_01X02, Pin_Headers:Pin_Header_Straight_1x02, F.Cu at (148.5, 105.0)
- added P5: CONN_02X04, UNCAMotorsports:MX120G-12, F.Cu at (148.5, 105.0)
- added Q1, Q2, Q3, Q5, Q6: Q_NMOS_GSD, TO_SOT_Packages_SMD:SOT-23_Handsoldering, F.Cu at (148.5, 105.0)
- added Q4: Q_PMOS_GSD, TO_SOT_Packages_SMD:SOT-23_Handsoldering, F.Cu at (148.5, 105.0)
- added R1, R10, R11, R12, R13, R14, R15, R16, R17, R18, R19, R21, R3, R31, R35, R36, R40, R41, R7, R8, R9: 10k, Resistors_SMD:R_0805_HandSoldering, F.Cu at (148.5, 105.0)
- added R2, R26, R4: 0R, Resistors_SMD:R_0805_HandSoldering, F.Cu at (148.5, 105.0)
- added R20, R28: 2.2k, Resistors_SMD:R_0805_HandSoldering, F.Cu at (148.5, 105.0)
- added R22, R23, R30, R33, R34: 220, Resistors_SMD:R_0805_HandSoldering, F.Cu at (148.5, 105.0)
- added R24: 330k, Resistors_SMD:R_0805_HandSoldering, F.Cu at (148.5, 105.0)
- added R25: 120k, Resistors_SMD:R_0805_HandSoldering, F.Cu at (148.5, 105.0)
- added R27, R5, R6: 620, Resistors_SMD:R_0805_HandSoldering, F.Cu at (148.5, 105.0)
- added R29, R39, R48: 470, Resistors_SMD:R_0805_HandSoldering, F.Cu at (148.5, 105.0)
- added R32: 120, Resistors_SMD:R_0805_HandSoldering, F.Cu at (148.5, 105.0)
- added R37, R38, R42, R43, R44, R45, R46, R47: 4.7k, Resistors_SMD:R_0805_HandSoldering, F.Cu at (148.5, 105.0)
- added U1, U2: BTS4130QGA, UNCAMotorsports:SOIC20-WIDE, F.Cu at (148.5, 105.0)
- added U10, U3, U4: BTS6133D, UNCAMotorsports:TO-252-5, F.Cu at (148.5, 105.0)
- added U11: R-78E5.0-1.0, UNCAMotorsports:R-78Cxx-1.0, F.Cu at (148.5, 105.0)
- added U12: FGMMOPA6H, UNCAMotorsports:GPS_16x16, F.Cu at (148.5, 105.0)
- added U13: U.FL_Antenna, UNCAMotorsports:U.FL-CON, F.Cu at (148.5, 105.0)
- added U14: NDC7002N, TO_SOT_Packages_SMD:SOT-23-6, F.Cu at (148.5, 105.0)
- added U15: MCP2551, SMD_Packages:SOIC-8-N, F.Cu at (148.5, 105.0)
- added U16: MC_Override, UNCAMotorsports:ALE1PB48, F.Cu at (148.5, 105.0)
- added U17: MCR_Shtdwn, UNCAMotorsports:ALE1PB48, F.Cu at (148.5, 105.0)
- added U18: MCL_Shtdwn, UNCAMotorsports:ALE1PB48, F.Cu at (148.5, 105.0)
- added U19: RI-0505S, UNCAMotorsports:RI-0505S, F.Cu at (148.5, 105.0)
- added U20: ISO1540, SMD_Packages:SOIC-8-N, F.Cu at (148.5, 105.0)
- added U21: TCMT1103, UNCAMotorsports:SSOP-4, F.Cu at (148.5, 105.0)
- added U22: OPTO-TRANSISTOR-4, UNCAMotorsports:SOIC16, F.Cu at (148.5, 105.0)
- added U23: PC_RLY, UNCAMotorsports:G6DN-1A, F.Cu at (148.5, 105.0)
- added U24: MCP47FEBX2, Housings_SSOP:TSSOP-8_4.4x3mm_Pitch0.65mm, F.Cu at (148.5, 105.0)
- added U5: H3LIS331DL, UNCAMotorsports:LGA-16-3x3, F.Cu at (148.5, 105.0)
- added U6: UltimateSensorFusion, UNCAMotorsports:UltimateSensorFusion, F.Cu at (148.5, 105.0)
- added U7: Teensy_3.5, UNCAMotorsports:Teensy_3.5, F.Cu at (148.5, 105.0)
- added U8: NDC7003P, TO_SOT_Packages_SMD:SOT-23-6, F.Cu at (148.5, 105.0)
- added U9: TL431, TO_SOT_Packages_SMD:SOT-23_Handsoldering, F.Cu at (148.5, 105.0)
Other:
- board outline added: 3.4 x 3.4 mm

Commit message: Small schematic fixes, start layout
Parts:
- added Q7: Q_NMOS_GSD, TO_SOT_Packages_SMD:SOT-23_Handsoldering, F.Cu at (211.6, 46.5)
- added R49: DNP, Resistors_SMD:R_0805_HandSoldering, F.Cu at (211.4, 43.5)
- added R50: DNP, Resistors_SMD:R_0805_HandSoldering, F.Cu at (211.4, 41.4)
- BT1, C7, C8: moved to B.Cu
- D11: value CANTX -> CANRX
- D12: value CANRX -> CANTX
- D13, D14, D15, D16, D17, D18, D5, D6: footprint Diodes_SMD:SMC_Handsoldering -> Diodes_SMD:SMA_Handsoldering
- U16: footprint UNCAMotorsports:ALE1PB48 -> UNCAMotorsports:G6DN-1A
- moved J9 139.5 mm to (20.1, 159.5), turned to 90 degrees
- moved R45 134.7 mm to (32.5, 173.5), turned to 180 degrees
- moved R44 133.5 mm to (32.5, 171.2), turned to 180 degrees
- moved J10 132.8 mm to (20.1, 138.8), turned to 90 degrees
- moved R43 132.4 mm to (32.5, 168.9), turned to 180 degrees
- moved R5 131.5 mm to (259.1, 33.8)
- moved R42 131.3 mm to (32.5, 166.6), turned to 180 degrees
- moved R2 130.3 mm to (259.1, 36.1)
- moved C1 129.6 mm to (267.5, 53.6)
- moved Q1 128.6 mm to (259.1, 39.4), turned to 270 degrees
- moved D17 128.5 mm to (20.3, 95.5), turned to 90 degrees
- moved D16 128.3 mm to (20.3, 109.7), turned to 90 degrees
- moved U5 127.4 mm to (267.5, 59.4), turned to 270 degrees
- moved U22 127.0 mm to (39.6, 170.3), turned to 270 degrees
- moved U24 126.7 mm to (28.9, 147.0), turned to 270 degrees
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Connections:
- R33 pad 1: +5V -> +3V3
- R34 pad 1: +5V -> +3V3
- U12 pad 13: /1PPS -> Net-(Q7-Pad1)
- U14 pad 1: /CANTX -> /CANRX
- U14 pad 3: /CANRX -> /CANTX
Routing:
- net GND: track 0.00 -> 129.6 mm, vias 0 -> 27
- net /GPS/VBACKUP: track 0.00 -> 33.0 mm, vias 0 -> 1
- net /CAN Bus/CANL: track 0.00 -> 28.3 mm
- net +3V3: track 0.00 -> 24.0 mm, vias 0 -> 7
- net /CAN Bus/CANH: track 0.00 -> 18.7 mm
- net +12V: track 0.00 -> 15.3 mm
- net +5VA: track 0.00 -> 14.2 mm
- net /CANRX: track 0.00 -> 12.8 mm, vias 0 -> 1
- net Net-(C7-Pad1): track 0.00 -> 11.2 mm
- net /Isolation/SDA_ISO: track 0.00 -> 10.4 mm, vias 0 -> 2
- net Net-(Q7-Pad1): track 0.00 -> 9.45 mm
- net Net-(D15-Pad1): track 0.00 -> 9.19 mm
- net /Isolation/SCL_ISO: track 0.00 -> 8.37 mm
- net +5V: track 0.00 -> 8.25 mm
- net Net-(D2-Pad1): track 0.00 -> 7.96 mm
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Other:
- copper layers 2 -> 4
- net class 3A added: clearance 0.3048, trace_width 0.6096, via_dia 1.016, via_drill 0.508
- net class Default: clearance 0.2 -> 0.2032; trace_width 0.25 -> 0.3048; via_dia 0.6 -> 0.8
- rule trace_clearance: 0.2 -> 0.2032
- rule trace_min: 0.2 -> 0.1524

Commit message: Major layout of VCU begins.  Moved some nets to facilitate layout
Parts:
- added TP1: TEST, Measurement_Points:Measurement_Point_Round-SMD-Pad_Big, F.Cu at (118.1, 141.0)
- added TP2: TEST, Measurement_Points:Measurement_Point_Round-SMD-Pad_Big, F.Cu at (123.2, 141.0)
- added TP3: TEST, Measurement_Points:Measurement_Point_Round-SMD-Pad_Big, F.Cu at (22.9, 141.0)
- added TP4: TEST, Measurement_Points:Measurement_Point_Round-SMD-Pad_Big, F.Cu at (27.9, 141.0)
- C4, D16, D17, R10, R11, R12, R13, R14, R15, R16, R17, R18, R22, R23, R42, R43, R44, R45, R7, R8, R9, U22, U8: moved to B.Cu
- moved R18 170.5 mm to (88.6, 125.6), turned to 0 degrees
- moved R14 168.7 mm to (88.6, 123.6), turned to 0 degrees
- moved R17 166.9 mm to (88.6, 121.5), turned to 0 degrees
- moved R16 165.2 mm to (88.6, 119.5), turned to 0 degrees
- moved U2 164.6 mm to (88.5, 120.5), turned to 270 degrees
- moved R13 163.5 mm to (88.6, 117.5), turned to 0 degrees
- moved R15 161.8 mm to (88.6, 115.4), turned to 0 degrees
- moved F8 158.6 mm to (99.3, 125.2), turned to 180 degrees
- moved F7 155.3 mm to (99.3, 121.7), turned to 180 degrees
- moved F6 152.0 mm to (99.3, 118.1), turned to 180 degrees
- moved F5 148.9 mm to (99.3, 114.6), turned to 180 degrees
- moved R12 146.7 mm to (88.6, 140.2), turned to 0 degrees
- moved R8 144.5 mm to (88.6, 137.9), turned to 0 degrees
- moved R11 142.3 mm to (88.6, 135.6), turned to 0 degrees
- moved P2 140.8 mm to (107.0, 107.0), turned to 270 degrees
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Connections:
- U7 pad 20: /5VOUT0 -> /Isolation/F_R2
- U7 pad 21: /5VOUT1 -> /Isolation/F_R1
- U7 pad 22: /5VOUT2 -> /Isolation/F_L2
- U7 pad 23: /5VOUT3 -> /Isolation/F_L1
- U7 pad 25: /Isolation/F_R2 -> /5VOUT3
- U7 pad 26: /Isolation/F_R1 -> /5VOUT2
- U7 pad 27: /Isolation/F_L2 -> /5VOUT1
- U7 pad 28: /Isolation/F_L1 -> /5VOUT0
Routing:
- net GND: track 129.6 -> 8.89 mm, vias 27 -> 0
- net /GPS/VBACKUP: track 33.0 -> 0.00 mm, vias 1 -> 0
- net /CAN Bus/CANL: track 28.3 -> 0.00 mm
- net +3V3: track 24.0 -> 2.20 mm, vias 7 -> 0
- net GNDA: track 0.00 -> 20.5 mm, vias 0 -> 1
- net /CAN Bus/CANH: track 18.7 -> 0.00 mm
- net +12V: track 15.3 -> 0.00 mm
- net /CANRX: track 12.8 -> 0.00 mm, vias 1 -> 0
- net Net-(D14-Pad2): track 0.00 -> 12.5 mm
- net /Isolation/CONTACT_R: track 0.00 -> 12.1 mm
- net Net-(C7-Pad1): track 11.2 -> 0.00 mm
- net Net-(Q7-Pad1): track 9.45 -> 0.00 mm
- net Net-(D15-Pad1): track 9.19 -> 0.00 mm
- net /Isolation/HV_BATT+: track 4.57 -> 13.8 mm
- net +5V: track 8.25 -> 16.2 mm, vias 0 -> 1
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- added copper zone on PWR, net +5V
- added copper zone on PWR, net +5VA
- added copper zone on GND, net GND
- added copper zone on GND, net GNDA
Other:
- board size 3.4 x 3.4 mm -> 127 x 68.6 mm

Commit message: VCU layout progress
Parts:
- C12, D1, D11, D12, J7, P4, P5, Q2, R3, R32, R33, R34, R4, R6, U14, U15, U4: moved to B.Cu
- moved J1 150.7 mm to (108.9, 81.0), turned to 180 degrees
- moved D7 121.3 mm to (115.1, 105.3)
- moved F10 121.3 mm to (118.9, 105.1)
- moved R24 121.3 mm to (108.7, 96.4)
- moved R26 121.3 mm to (108.7, 101.7)
- moved U11 121.3 mm to (118.9, 96.1)
- moved U9 121.3 mm to (105.7, 91.2)
- moved C6 121.3 mm to (106.2, 101.7)
- moved C7 121.3 mm to (115.6, 98.4)
- moved C8 121.3 mm to (115.6, 93.6)
- moved D9 121.3 mm to (118.4, 88.6)
- moved R25 121.3 mm to (106.2, 96.4)
- moved R29 121.3 mm to (113.7, 88.6)
- moved F9 119.5 mm to (135.4, 90.4)
- moved R28 119.5 mm to (129.5, 107.2)
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Connections:
- J1 pad 10: Net-(J1-Pad10) -> (no net)
- J1 pad 12: Net-(J1-Pad12) -> (no net)
- U12 pad 14: Net-(U12-Pad14) -> (no net)
- U12 pad 15: Net-(U12-Pad15) -> (no net)
- U12 pad 16: Net-(U12-Pad16) -> (no net)
- U12 pad 17: Net-(U12-Pad17) -> (no net)
- U12 pad 18: Net-(U12-Pad18) -> (no net)
- U12 pad 20: Net-(U12-Pad20) -> (no net)
- U12 pad 6: Net-(U12-Pad6) -> (no net)
- U12 pad 7: Net-(U12-Pad7) -> (no net)
- U15 pad 5: Net-(U15-Pad5) -> (no net)
- U22 pad 2: GND -> GNDA
- U22 pad 4: GND -> GNDA
- U22 pad 6: GND -> GNDA
- U22 pad 8: GND -> GNDA
- U24 pad 2: Net-(U24-Pad2) -> (no net)
- U5 pad 2: Net-(U5-Pad2) -> (no net)
- U5 pad 3: Net-(U5-Pad3) -> (no net)
- U6 pad 3: Net-(U6-Pad3) -> (no net)
- U7 pad 32: Net-(U7-Pad32) -> (no net)
- U7 pad 33: Net-(U7-Pad33) -> (no net)
- U7 pad 35: Net-(U7-Pad35) -> (no net)
- U7 pad 43: Net-(U7-Pad43) -> (no net)
- U7 pad 44: Net-(U7-Pad44) -> (no net)
- U7 pad 45: Net-(U7-Pad45) -> (no net)
- U7 pad 47: Net-(U7-Pad47) -> (no net)
Routing:
- net +12V: track 0.00 -> 138.4 mm, vias 0 -> 9
- net GND: track 8.89 -> 127.6 mm, vias 0 -> 23
- net /Isolation/KSI: track 0.00 -> 92.7 mm
- net +3V3: track 2.20 -> 73.6 mm, vias 0 -> 2
- net /GLV_CURRENT: track 0.00 -> 55.0 mm
- net /AMS_F_OUT: track 0.00 -> 53.3 mm, vias 0 -> 1
- net /SHTDWN_CURRENT: track 0.00 -> 52.0 mm
- net /SDA1: track 2.90 -> 49.7 mm, vias 0 -> 3
- net /Isolation/FAULT_L1: track 0.00 -> 46.8 mm, vias 0 -> 5
- net /Isolation/FAULT_L2: track 0.00 -> 43.8 mm, vias 0 -> 1
- net /SCL1: track 2.69 -> 46.2 mm
- net /Isolation/DAC_L: track 0.00 -> 43.4 mm
- net /IMD_F_OUT: track 0.00 -> 43.4 mm, vias 0 -> 2
- net /BRAKE_IN: track 0.00 -> 40.5 mm
- net /CAN Bus/CANH: track 0.00 -> 38.1 mm
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