File: VehicleController/file58B363B0.sch (KiCad schematic (older format))
At the start: 11 parts, among them J7 CAN_SER, P4 CONN_01X02, P5 CONN_02X04, U14 NDC7002N, U15 MCP2551

Commit message: Re-do MX120, GDS->GSD, Associations.
Parts:
- J7: footprint (none) -> Pin_Headers:Pin_Header_Straight_1x03_Pitch2.54mm
- P5: footprint (none) -> UNCA Motorsports:MX120G-12
Changed lines of the file:
@@
 $EndComp
 $Comp
-L GND #PWR61
+L GND #PWR056
 U 1 1 58B3658D
 P 5950 3500
-F 0 "#PWR61" H 5950 3250 50  0001 C CNN
+F 0 "#PWR056" H 5950 3250 50  0001 C CNN
 F 1 "GND" H 5955 3327 50  0000 C CNN
 F 2 "" H 5950 3500 50  0000 C CNN
@@
 NoConn ~ 5850 3050
 $Comp
-L +5V #PWR59
+L +5V #PWR057
 U 1 1 58B36594
 P 4900 2950
-F 0 "#PWR59" H 4900 2800 50  0001 C CNN
+F 0 "#PWR057" H 4900 2800 50  0001 C CNN
 F 1 "+5V" H 4915 3123 50  0000 C CNN
 F 2 "" H 4900 2950 50  0000 C CNN
@@
 $EndComp
 $Comp
-L GND #PWR60
+L GND #PWR058
 U 1 1 58B3659A
 P 4950 3500
-F 0 "#PWR60" H 4950 3250 50  0001 C CNN
+F 0 "#PWR058" H 4950 3250 50  0001 C CNN
 F 1 "GND" H 4955 3327 50  0000 C CNN
 F 2 "" H 4950 3500 50  0000 C CNN
@@
 $EndComp
 $Comp
-L +5V #PWR56
+L +5V #PWR059
 U 1 1 58B0DEC8
 P 4250 3000
-F 0 "#PWR56" H 4250 2850 50  0001 C CNN
+F 0 "#PWR059" H 4250 2850 50  0001 C CNN
 F 1 "+5V" H 4265 3173 50  0000 C CNN
 F 2 "" H 4250 3000 50  0000 C CNN
@@
 $EndComp
 $Comp
-L GND #PWR57
+L GND #PWR060
 U 1 1 58B0DF2A
 P 4250 3450
-F 0 "#PWR57" H 4250 3200 50  0001 C CNN
+F 0 "#PWR060" H 4250 3200 50  0001 C CNN
 F 1 "GND" H 4255 3277 50  0000 C CNN
 F 2 "" H 4250 3450 50  0000 C CNN
@@
 	7000 3050 7100 3050
 $Comp
-L GND #PWR64
+L GND #PWR061
 U 1 1 58B7F609
 P 7000 3450
-F 0 "#PWR64" H 7000 3200 50  0001 C CNN
+F 0 "#PWR061" H 7000 3200 50  0001 C CNN
 F 1 "GND" H 7005 3277 50  0000 C CNN
 F 2 "" H 7000 3450 50  0000 C CNN
@@
 	7700 3050 7700 2950
 $Comp
-L GND #PWR66
+L GND #PWR062
 U 1 1 58B7FA08
 P 7700 3450
-F 0 "#PWR66" H 7700 3200 50  0001 C CNN
+F 0 "#PWR062" H 7700 3200 50  0001 C CNN
 F 1 "GND" H 7705 3277 50  0000 C CNN
 F 2 "" H 7700 3450 50  0000 C CNN
@@
 	7700 3350 7700 3450
 $Comp
-L +12V #PWR63
+L +12V #PWR063
 U 1 1 58BABA64
 P 7000 2950
-F 0 "#PWR63" H 7000 2800 50  0001 C CNN
+F 0 "#PWR063" H 7000 2800 50  0001 C CNN
 F 1 "+12V" H 7015 3123 50  0000 C CNN
 F 2 "" H 7000 2950 50  0000 C CNN
@@
 $EndComp
 $Comp
-L +12V #PWR65
+L +12V #PWR064
 U 1 1 58BABA85
 P 7700 2950
-F 0 "#PWR65" H 7700 2800 50  0001 C CNN
+F 0 "#PWR064" H 7700 2800 50  0001 C CNN
 F 1 "+12V" H 7715 3123 50  0000 C CNN
 F 2 "" H 7700 2950 50  0000 C CNN
@@
 	4600 4700 4800 4700
 $Comp
-L GND #PWR58
+L GND #PWR065
 U 1 1 58C2C777
 P 4700 5000
-F 0 "#PWR58" H 1200 2500 50  0001 C CNN
+F 0 "#PWR065" H 1200 2500 50  0001 C CNN
 F 1 "GND" H 4705 4827 50  0000 C CNN
 F 2 "" H 1200 2750 50  0001 C CNN
@@
 	5750 4850 5950 4850
 $Comp
-L +5V #PWR62
+L +5V #PWR066
 U 1 1 58C2D6D1
 P 6350 4450
-F 0 "#PWR62" H 850 2600 50  0001 C CNN
+F 0 "#PWR066" H 850 2600 50  0001 C CNN
 F 1 "+5V" H 6365 4623 50  0000 C CNN
 F 2 "" H 850 2750 50  0001 C CNN
@@
 F 0 "P5" H 7350 3450 50  0000 C CNN
 F 1 "CONN_02X04" H 7350 2950 50  0000 C CNN
-F 2 "" H 7350 2000 50  0001 C CNN
+F 2 "UNCA Motorsports:MX120G-12" H 7350 2000 50  0001 C CNN
 F 3 "" H 7350 2000 50  0000 C CNN
 	1    7350 3200
@@
 F 0 "J7" H 3100 3400 50  0000 C CNN
 F 1 "CAN_SER" V 3200 3200 50  0000 C CNN
-F 2 "" H 3100 3200 50  0001 C CNN
+F 2 "Pin_Headers:Pin_Header_Straight_1x03_Pitch2.54mm" H 3100 3200 50  0001 C CNN
 F 3 "" H 3100 3200 50  0001 C CNN
 	1    3100 3200
@@
 CANRX
 $Comp
-L GND #PWR55
+L GND #PWR067
 U 1 1 59121912
 P 3450 3400
-F 0 "#PWR55" H 3450 3150 50  0001 C CNN
+F 0 "#PWR067" H 3450 3150 50  0001 C CNN
 F 1 "GND" H 3455 3227 50  0000 C CNN
 F 2 "" H 3450 3400 50  0000 C CNN

Commit message: Library Fixes
Parts:
- J7: footprint Pin_Headers:Pin_Header_Straight_1x03_Pitch2.54mm -> Pin_Headers:Pin_Header_Straight_1x03
- P4: footprint Pin_Headers:Pin_Header_Angled_1x02 -> Pin_Headers:Pin_Header_Straight_1x02
- P5: footprint UNCA Motorsports:MX120G-12 -> UNCAMotorsports:MX120G-12
Changed lines of the file:
@@
 F 0 "P4" V 5765 2245 50  0000 C CNN
 F 1 "CONN_01X02" V 5674 2245 50  0000 C CNN
-F 2 "Pin_Headers:Pin_Header_Angled_1x02" H 5550 2250 50  0001 C CNN
+F 2 "Pin_Headers:Pin_Header_Straight_1x02" H 5550 2250 50  0001 C CNN
 F 3 "" H 5550 2250 50  0000 C CNN
 	1    5550 2250
@@
 F 0 "P5" H 7350 3450 50  0000 C CNN
 F 1 "CONN_02X04" H 7350 2950 50  0000 C CNN
-F 2 "UNCA Motorsports:MX120G-12" H 7350 2000 50  0001 C CNN
+F 2 "UNCAMotorsports:MX120G-12" H 7350 2000 50  0001 C CNN
 F 3 "" H 7350 2000 50  0000 C CNN
 	1    7350 3200
@@
 F 0 "J7" H 3100 3400 50  0000 C CNN
 F 1 "CAN_SER" V 3200 3200 50  0000 C CNN
-F 2 "Pin_Headers:Pin_Header_Straight_1x03_Pitch2.54mm" H 3100 3200 50  0001 C CNN
+F 2 "Pin_Headers:Pin_Header_Straight_1x03" H 3100 3200 50  0001 C CNN
 F 3 "" H 3100 3200 50  0001 C CNN
 	1    3100 3200

Commit message: Small schematic fixes, start layout
Parts:
- D11: value CANTX -> CANRX
- D12: value CANRX -> CANTX
Connections:
- net +5V: no longer R33.1, R34.1
- net CANRX: now also U14.1 (G1); no longer U14.3 (G2)
- net CANTX: now also U14.3 (G2); no longer U14.1 (G1)
- new net +3V3: R33.1, R34.1
Changed lines of the file:
@@
 LIBS:VehicleController-rescue
 LIBS:UNCAMotorsports
-LIBS:power
-LIBS:device
-LIBS:transistors
-LIBS:conn
-LIBS:linear
-LIBS:regul
-LIBS:74xx
-LIBS:cmos4000
-LIBS:adc-dac
-LIBS:memory
-LIBS:xilinx
-LIBS:microcontrollers
-LIBS:dsp
-LIBS:microchip
-LIBS:analog_switches
-LIBS:motorola
-LIBS:texas
-LIBS:intel
-LIBS:audio
-LIBS:interface
-LIBS:digital-audio
-LIBS:philips
-LIBS:display
-LIBS:cypress
-LIBS:siliconi
-LIBS:opto
-LIBS:atmel
-LIBS:contrib
-LIBS:valves
 LIBS:Common-Parts-Library-CPL
 LIBS:relays
 LIBS:SystemBlocks
-LIBS:dc-dc
-LIBS:Power_Management
-LIBS:switches
 LIBS:VehicleController-cache
-EELAYER 25 0
+EELAYER 26 0
 EELAYER END
 $Descr A4 11693 8268
@@
 $EndComp
 $Comp
-L GND #PWR056
+L GND #PWR057
 U 1 1 58B3658D
 P 5950 3500
-F 0 "#PWR056" H 5950 3250 50  0001 C CNN
+F 0 "#PWR057" H 5950 3250 50  0001 C CNN
 F 1 "GND" H 5955 3327 50  0000 C CNN
 F 2 "" H 5950 3500 50  0000 C CNN
@@
 NoConn ~ 5850 3050
 $Comp
-L +5V #PWR057
+L +5V #PWR058
 U 1 1 58B36594
 P 4900 2950
-F 0 "#PWR057" H 4900 2800 50  0001 C CNN
+F 0 "#PWR058" H 4900 2800 50  0001 C CNN
 F 1 "+5V" H 4915 3123 50  0000 C CNN
 F 2 "" H 4900 2950 50  0000 C CNN
@@
 $EndComp
 $Comp
-L GND #PWR058
+L GND #PWR059
 U 1 1 58B3659A
 P 4950 3500
-F 0 "#PWR058" H 4950 3250 50  0001 C CNN
+F 0 "#PWR059" H 4950 3250 50  0001 C CNN
 F 1 "GND" H 4955 3327 50  0000 C CNN
 F 2 "" H 4950 3500 50  0000 C CNN
@@
 $EndComp
 $Comp
-L +5V #PWR059
+L +5V #PWR060
 U 1 1 58B0DEC8
 P 4250 3000
-F 0 "#PWR059" H 4250 2850 50  0001 C CNN
+F 0 "#PWR060" H 4250 2850 50  0001 C CNN
 F 1 "+5V" H 4265 3173 50  0000 C CNN
 F 2 "" H 4250 3000 50  0000 C CNN
@@
 $EndComp
 $Comp
-L GND #PWR060
+L GND #PWR061
 U 1 1 58B0DF2A
 P 4250 3450
-F 0 "#PWR060" H 4250 3200 50  0001 C CNN
+F 0 "#PWR061" H 4250 3200 50  0001 C CNN
 F 1 "GND" H 4255 3277 50  0000 C CNN
 F 2 "" H 4250 3450 50  0000 C CNN
@@
 	7000 3050 7100 3050
 $Comp
-L GND #PWR061
+L GND #PWR062
 U 1 1 58B7F609
 P 7000 3450
-F 0 "#PWR061" H 7000 3200 50  0001 C CNN
+F 0 "#PWR062" H 7000 3200 50  0001 C CNN
 F 1 "GND" H 7005 3277 50  0000 C CNN
 F 2 "" H 7000 3450 50  0000 C CNN
@@
 	7700 3050 7700 2950
 $Comp
-L GND #PWR062
+L GND #PWR063
 U 1 1 58B7FA08
 P 7700 3450
-F 0 "#PWR062" H 7700 3200 50  0001 C CNN
+F 0 "#PWR063" H 7700 3200 50  0001 C CNN
 F 1 "GND" H 7705 3277 50  0000 C CNN
 F 2 "" H 7700 3450 50  0000 C CNN
@@
 	7700 3350 7700 3450
 $Comp
-L +12V #PWR063
+L +12V #PWR064
 U 1 1 58BABA64
 P 7000 2950
-F 0 "#PWR063" H 7000 2800 50  0001 C CNN
+F 0 "#PWR064" H 7000 2800 50  0001 C CNN
 F 1 "+12V" H 7015 3123 50  0000 C CNN
 F 2 "" H 7000 2950 50  0000 C CNN
@@
 $EndComp
 $Comp
-L +12V #PWR064
+L +12V #PWR065
 U 1 1 58BABA85
 P 7700 2950
-F 0 "#PWR064" H 7700 2800 50  0001 C CNN
+F 0 "#PWR065" H 7700 2800 50  0001 C CNN
 F 1 "+12V" H 7715 3123 50  0000 C CNN
 F 2 "" H 7700 2950 50  0000 C CNN
@@
 	1    0    0    -1
 $EndComp
+Text HLabel 4600 4700 0    60   Input ~ 0
+CANTX
 Text HLabel 4600 4600 0    60   Input ~ 0
-CANTX
-Text HLabel 4600 4700 0    60   Input ~ 0
 CANRX
 Wire Wire Line
+	4600 4700 4800 4700
+Wire Wire Line
 	4600 4600 4800 4600
-Wire Wire Line
-	4600 4700 4800 4700
-$Comp
-L GND #PWR065
+$Comp
+L GND #PWR066
 U 1 1 58C2C777
 P 4700 5000
-F 0 "#PWR065" H 1200 2500 50  0001 C CNN
+F 0 "#PWR066" H 1200 2500 50  0001 C CNN
 F 1 "GND" H 4705 4827 50  0000 C CNN
 F 2 "" H 1200 2750 50  0001 C CNN
@@
 P 5650 4650
 F 0 "D11" H 5650 4885 50  0000 C CNN
-F 1 "CANTX" H 5650 4794 50  0000 C CNN
+F 1 "CANRX" H 5650 4794 50  0000 C CNN
 F 2 "LEDs:LED-0805" V 1100 3550 50  0001 C CNN
 F 3 "" V 1100 3550 50  0001 C CNN
@@
 P 5650 4850
 F 0 "D12" H 5650 4650 50  0000 C CNN
-F 1 "CANRX" H 5650 4750 50  0000 C CNN
+F 1 "CANTX" H 5650 4750 50  0000 C CNN
 F 2 "LEDs:LED-0805" V 1100 3750 50  0001 C CNN
 F 3 "" V 1100 3750 50  0001 C CNN
@@
 Wire Wire Line
 	5750 4850 5950 4850
-$Comp
-L +5V #PWR066
-U 1 1 58C2D6D1
-P 6350 4450
-F 0 "#PWR066" H 850 2600 50  0001 C CNN
-F 1 "+5V" H 6365 4623 50  0000 C CNN
-F 2 "" H 850 2750 50  0001 C CNN
-F 3 "" H 850 2750 50  0001 C CNN
-	1    6350 4450
-	1    0    0    -1
-$EndComp
 Wire Wire Line
 	6150 4650 6350 4650
@@
 Wire Wire Line
 	3300 3100 3500 3100
+$Comp
+L +3V3 #PWR068
+U 1 1 5919DAF9
+P 6350 4450
+F 0 "#PWR068" H 6350 4300 50  0001 C CNN
+F 1 "+3V3" H 6365 4623 50  0000 C CNN
+F 2 "" H 6350 4450 50  0001 C CNN
+F 3 "" H 6350 4450 50  0001 C CNN
+	1    6350 4450
+	1    0    0    -1
+$EndComp
 $EndSCHEMATC

Commit message: More VCU layout work
connectors changed to 2x4 molex nanofits for the 12v and 5v outputs.
Parts:
- P5: footprint UNCAMotorsports:MX120G-12 -> Connectors_Molex:Molex_NanoFit_2x04x2.50mm_Straight
Changed lines of the file:
@@
 F 0 "P5" H 7350 3450 50  0000 C CNN
 F 1 "CONN_02X04" H 7350 2950 50  0000 C CNN
-F 2 "UNCAMotorsports:MX120G-12" H 7350 2000 50  0001 C CNN
+F 2 "Connectors_Molex:Molex_NanoFit_2x04x2.50mm_Straight" H 7350 2000 50  0001 C CNN
 F 3 "" H 7350 2000 50  0000 C CNN
 	1    7350 3200

Commit message: Major VCU Layout changes
Connections:
- net CANRX: now also U14.3 (G2); no longer U14.1 (G1)
- net CANTX: now also U14.1 (G1); no longer U14.3 (G2)
Changed lines of the file:
@@
 $EndComp
 $Comp
-L GND #PWR060
+L GND #PWR059
 U 1 1 58B3658D
 P 5950 3500
-F 0 "#PWR060" H 5950 3250 50  0001 C CNN
+F 0 "#PWR059" H 5950 3250 50  0001 C CNN
 F 1 "GND" H 5955 3327 50  0000 C CNN
 F 2 "" H 5950 3500 50  0000 C CNN
@@
 NoConn ~ 5850 3050
 $Comp
-L +5V #PWR061
+L +5V #PWR060
 U 1 1 58B36594
 P 4900 2950
-F 0 "#PWR061" H 4900 2800 50  0001 C CNN
+F 0 "#PWR060" H 4900 2800 50  0001 C CNN
 F 1 "+5V" H 4915 3123 50  0000 C CNN
 F 2 "" H 4900 2950 50  0000 C CNN
@@
 $EndComp
 $Comp
-L GND #PWR062
+L GND #PWR061
 U 1 1 58B3659A
 P 4950 3500
-F 0 "#PWR062" H 4950 3250 50  0001 C CNN
+F 0 "#PWR061" H 4950 3250 50  0001 C CNN
 F 1 "GND" H 4955 3327 50  0000 C CNN
 F 2 "" H 4950 3500 50  0000 C CNN
@@
 $EndComp
 $Comp
-L +5V #PWR063
+L +5V #PWR062
 U 1 1 58B0DEC8
 P 4250 3000
-F 0 "#PWR063" H 4250 2850 50  0001 C CNN
+F 0 "#PWR062" H 4250 2850 50  0001 C CNN
 F 1 "+5V" H 4265 3173 50  0000 C CNN
 F 2 "" H 4250 3000 50  0000 C CNN
@@
 $EndComp
 $Comp
-L GND #PWR064
+L GND #PWR063
 U 1 1 58B0DF2A
 P 4250 3450
-F 0 "#PWR064" H 4250 3200 50  0001 C CNN
+F 0 "#PWR063" H 4250 3200 50  0001 C CNN
 F 1 "GND" H 4255 3277 50  0000 C CNN
 F 2 "" H 4250 3450 50  0000 C CNN
@@
 	7000 3050 7100 3050
 $Comp
-L GND #PWR065
+L GND #PWR064
 U 1 1 58B7F609
 P 7000 3450
-F 0 "#PWR065" H 7000 3200 50  0001 C CNN
+F 0 "#PWR064" H 7000 3200 50  0001 C CNN
 F 1 "GND" H 7005 3277 50  0000 C CNN
 F 2 "" H 7000 3450 50  0000 C CNN
@@
 	7700 3050 7700 2950
 $Comp
-L GND #PWR066
+L GND #PWR065
 U 1 1 58B7FA08
 P 7700 3450
-F 0 "#PWR066" H 7700 3200 50  0001 C CNN
+F 0 "#PWR065" H 7700 3200 50  0001 C CNN
 F 1 "GND" H 7705 3277 50  0000 C CNN
 F 2 "" H 7700 3450 50  0000 C CNN
@@
 	7700 3350 7700 3450
 $Comp
-L +12V #PWR067
+L +12V #PWR066
 U 1 1 58BABA64
 P 7000 2950
-F 0 "#PWR067" H 7000 2800 50  0001 C CNN
+F 0 "#PWR066" H 7000 2800 50  0001 C CNN
 F 1 "+12V" H 7015 3123 50  0000 C CNN
 F 2 "" H 7000 2950 50  0000 C CNN
@@
 $EndComp
 $Comp
-L +12V #PWR068
+L +12V #PWR067
 U 1 1 58BABA85
 P 7700 2950
-F 0 "#PWR068" H 7700 2800 50  0001 C CNN
+F 0 "#PWR067" H 7700 2800 50  0001 C CNN
 F 1 "+12V" H 7715 3123 50  0000 C CNN
 F 2 "" H 7700 2950 50  0000 C CNN
@@
 	1    0    0    -1
 $EndComp
+Text HLabel 4600 4600 0    60   Input ~ 0
+CANTX
 Text HLabel 4600 4700 0    60   Input ~ 0
-CANTX
-Text HLabel 4600 4600 0    60   Input ~ 0
 CANRX
 Wire Wire Line
+	4600 4600 4800 4600
+Wire Wire Line
 	4600 4700 4800 4700
-Wire Wire Line
-	4600 4600 4800 4600
-$Comp
-L GND #PWR069
+$Comp
+L GND #PWR068
 U 1 1 58C2C777
 P 4700 5000
-F 0 "#PWR069" H 1200 2500 50  0001 C CNN
+F 0 "#PWR068" H 1200 2500 50  0001 C CNN
 F 1 "GND" H 4705 4827 50  0000 C CNN
 F 2 "" H 1200 2750 50  0001 C CNN
@@
 CANRX
 $Comp
-L GND #PWR070
+L GND #PWR069
 U 1 1 59121912
 P 3450 3400
-F 0 "#PWR070" H 3450 3150 50  0001 C CNN
+F 0 "#PWR069" H 3450 3150 50  0001 C CNN
 F 1 "GND" H 3455 3227 50  0000 C CNN
 F 2 "" H 3450 3400 50  0000 C CNN
@@
 	3300 3100 3500 3100
 $Comp
-L +3V3 #PWR071
+L +3V3 #PWR070
 U 1 1 5919DAF9
 P 6350 4450
-F 0 "#PWR071" H 6350 4300 50  0001 C CNN
+F 0 "#PWR070" H 6350 4300 50  0001 C CNN
 F 1 "+3V3" H 6365 4623 50  0000 C CNN
 F 2 "" H 6350 4450 50  0001 C CNN
