File: VehicleController/VehicleController.sch (KiCad schematic (older format))
At the start: 58 parts, among them J1 CONN_02X05, J2 USF_SLAVE_I2C, J3 USB_A, J4 USB_A, J5 I2C_0, J6 I2C_1, P1 OUTPUTS, P2 OUTPUTS, Q1 Q_NMOS_GSD, Q2 Q_NMOS_GSD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

Commit message: Finish VCU 4 layer
Connections:
- net SHTDWN_OUT is gone; now on net SHUTDOWN_OUT: J1.4 (P4)
- net AIR+: now also J1.9 (P9); no longer J1.8 (P8)
- net AMS_F_OUT: now also J1.3 (P3); no longer J1.10 (P10)
- net GLVMS: now also J1.10 (P10); no longer J1.3 (P3)
- net GLV_CURRENT: now also U7.35 ((SCK0)/13); no longer U7.36 ((PWM)A0/14)
- net IMD_F_OUT: now also J1.2 (P2); no longer J1.9 (P9)
- net TSMS: now also J1.8 (P8); no longer J1.2 (P2)
- net F_L2: now reaches U7.37 ((CS0)A1/15)
- net F_R1: now reaches U7.38 (A2/16)
- net F_R2: now reaches U7.39 (A3/17)
- net MC_OVERRIDE: no longer names the net of U7.26 ((RX5)A15/34)
- net MC_SHUTDOWN renamed SHUTDOWN_OUT
- new net F_L1: U7.36 ((PWM)A0/14)
- no-connect marks 7 -> 9
Changed lines of the file:
@@
 	-1   0    0    -1
 $EndComp
-Text Label 12400 4000 2    60   ~ 0
+Text Label 12400 4100 2    60   ~ 0
 GLV_CURRENT
 Text Label 12400 4600 2    60   ~ 0
@@
 L GND #PWR012
 U 1 1 58BAD6C3
-P 1100 2150
-F 0 "#PWR012" H 1100 1900 50  0001 C CNN
-F 1 "GND" H 1105 1977 50  0000 C CNN
-F 2 "" H 1100 2150 50  0000 C CNN
-F 3 "" H 1100 2150 50  0000 C CNN
-	1    1100 2150
-	-1   0    0    -1
-$EndComp
-Text Label 2450 2050 2    60   ~ 0
-SHTDWN_OUT
-Text Label 15850 5000 2    60   ~ 0
-SHTDWN_OUT
+P 650 2200
+F 0 "#PWR012" H 650 1950 50  0001 C CNN
+F 1 "GND" H 655 2027 50  0000 C CNN
+F 2 "" H 650 2200 50  0000 C CNN
+F 3 "" H 650 2200 50  0000 C CNN
+	1    650  2200
+	-1   0    0    -1
+$EndComp
+Text Label 2500 2050 2    60   ~ 0
+SHUTDOWN_OUT
 Text Label 2250 2950 0    60   ~ 0
 GLVMS
 Text Label 4350 2950 2    60   ~ 0
-MC_SHUTDOWN
-Text Label 15850 4900 2    60   ~ 0
-MC_SHUTDOWN
-Text Label 750  2050 0    60   ~ 0
+SHUTDOWN_OUT
+Text Label 2500 2350 2    60   ~ 0
 GLVMS
 Text Label 8950 2900 0    60   ~ 0
@@
 Text Label 8950 3500 0    60   ~ 0
 1PPS
-NoConn ~ 11750 4100
 $Comp
 L +3.3V #PWR013
@@
 Text Notes 9950 850  0    60   ~ 0
 Run USB from Teensy to J1, and J2 to exterior
-Text Label 2450 2150 2    60   ~ 0
+Text Label 2500 2150 2    60   ~ 0
 START_CAR
-Text Label 750  2250 0    60   ~ 0
+Text Label 850  2250 0    60   ~ 0
 BRAKE_IN
 Text Label 8950 3400 0    60   ~ 0
@@
 $EndComp
 NoConn ~ 11750 3300
-Text Label 850  2350 0    60   ~ 0
+Text Label 2500 1950 2    60   ~ 0
 IMD_F_OUT
-Text Label 2450 2350 2    60   ~ 0
+Text Label 850  2050 0    60   ~ 0
 AMS_F_OUT
-Text Label 2450 1950 2    60   ~ 0
+Text Label 2500 2250 2    60   ~ 0
 TSMS
 $Comp
@@
 	1    0    0    -1
 $EndComp
-Text Label 2450 2250 2    60   ~ 0
+Text Label 850  2350 0    60   ~ 0
 AIR+
 Text Notes 2650 4600 0    60   ~ 0
 Gets power from TSMS,\ndirectly controls TS+ AIR
-Text Label 15850 5150 2    60   ~ 0
-MC_OVERRIDE
-Text Label 12400 5000 2    60   ~ 0
-MC_OVERRIDE
 Text Label 14100 6500 0    60   ~ 0
 SCL0
@@
 Wire Wire Line
 	3650 3050 3650 2950
-Wire Wire Line
-	12400 5000 11750 5000
-Wire Wire Line
-	15050 5150 15850 5150
 Connection ~ 3650 4850
 Wire Wire Line
-	2450 2250 1850 2250
+	850  2350 1350 2350
 Connection ~ 2650 3500
 Wire Wire Line
@@
 	2400 3250 2400 3150
 Wire Wire Line
-	1850 1950 2450 1950
-Wire Wire Line
-	2450 2350 1850 2350
+	1850 2250 2500 2250
+Wire Wire Line
+	1350 2050 850  2050
 Wire Wire Line
 	2700 7450 2800 7450
@@
 	9550 3400 8950 3400
 Wire Wire Line
-	850  2350 1350 2350
-Wire Wire Line
-	1350 2250 750  2250
-Wire Wire Line
-	1850 2150 2450 2150
+	2500 1950 1850 1950
+Wire Wire Line
+	1350 2250 850  2250
+Wire Wire Line
+	1850 2150 2500 2150
 Connection ~ 11100 1900
 Wire Wire Line
@@
 	11750 4200 12050 4200
 Wire Wire Line
-	750  2050 1350 2050
-Wire Wire Line
-	15050 4900 15850 4900
+	2500 2350 1850 2350
 Wire Wire Line
 	2750 2950 2250 2950
 Wire Wire Line
-	15050 5000 15850 5000
-Wire Wire Line
-	1850 2050 2450 2050
+	1850 2050 2500 2050
 Wire Wire Line
 	850  950  850  850
@@
 	7800 3600 9550 3600
 Wire Wire Line
-	12400 4000 11750 4000
+	12400 4100 11750 4100
 Wire Wire Line
 	11600 9150 11000 9150
@@
 	650  2150 1350 2150
 Wire Wire Line
-	650  2150 650  2050
-Connection ~ 1100 2150
+	650  2050 650  2200
+Connection ~ 650  2150
 $Sheet
 S 13650 4400 1400 900
@@
 F3 "SCL_IN" I L 13650 4700 60
 F4 "DAC_LATCH" I L 13650 4500 60
-F5 "Shutdown_In" I R 15050 4900 60
-F6 "Shutdown_Out" O R 15050 5000 60
-F7 "PRECHARGE" I R 15050 4750 60
-F8 "+5V" I R 15050 4500 60
-F9 "TSMS" I R 15050 4650 60
-F10 "F_L1" O L 13650 5100 60
-F11 "F_L2" O L 13650 5000 60
-F12 "F_R1" O L 13650 4900 60
-F13 "F_R2" O L 13650 4800 60
-F14 "MC_OVERRIDE" I R 15050 5150 60
+F5 "PRECHARGE" I R 15050 4750 60
+F6 "+5V" I R 15050 4500 60
+F7 "TSMS" I R 15050 4650 60
+F8 "F_L1" O L 13650 5100 60
+F9 "F_L2" O L 13650 5000 60
+F10 "F_R1" O L 13650 4900 60
+F11 "F_R2" O L 13650 4800 60
 $EndSheet
 $Comp
@@
 Text Label 12050 4200 2    60   ~ 0
 GND
-NoConn ~ 11750 3900
+Wire Wire Line
+	13650 4800 13150 4800
+Text Label 13150 4800 0    60   ~ 0
+F_R2
+Text Label 13150 4900 0    60   ~ 0
+F_R1
+Text Label 13150 5000 0    60   ~ 0
+F_L2
+Text Label 13150 5100 0    60   ~ 0
+F_L1
+Wire Wire Line
+	13150 4900 13650 4900
+Wire Wire Line
+	13150 5000 13650 5000
+Wire Wire Line
+	13150 5100 13650 5100
+Wire Wire Line
+	11750 3700 12250 3700
+Text Label 12250 3700 2    60   ~ 0
+F_R2
+Text Label 12250 3800 2    60   ~ 0
+F_R1
+Text Label 12250 3900 2    60   ~ 0
+F_L2
+Text Label 12250 4000 2    60   ~ 0
+F_L1
+Wire Wire Line
+	12250 3800 11750 3800
+Wire Wire Line
+	12250 3900 11750 3900
+Wire Wire Line
+	12250 4000 11750 4000
+NoConn ~ 9550 3000
+NoConn ~ 9550 3100
+NoConn ~ 11750 3400
+NoConn ~ 11750 5000
 $EndSCHEMATC
