File: Brake System Plausibility Device/bspd.sch (KiCad schematic (older format))
At the start: 34 parts, among them P1 MX150_16, SW1 SW_Push, U1 MCP604, U2 LM1117-5.0, U3 74LVC2G74, U4 74AUC2G00, U5 L01Z400S05, U6 L01Z400S05

Commit message: BSPD Layout Done
Parts:
- removed P1: MX150_16, UNCAMotorsports:MX150_16pin, symbol MX150_16
- removed R12, R13: 10k, symbol R
- removed U5, U6: L01Z400S05, symbol L01Z400S05
- added J1: CURRENT_SENSE_1, Pin_Headers:Pin_Header_Straight_1x03_Pitch2.54mm, symbol CONN_01X03
- added J2: CURRENT_SENSE_2, Pin_Headers:Pin_Header_Straight_1x03_Pitch2.54mm, symbol CONN_01X03
- added J3: BRAKE_SENSOR, Pin_Headers:Pin_Header_Straight_1x03_Pitch2.54mm, symbol CONN_01X03
- added J4: 12V_AND_GND, Pin_Headers:Pin_Header_Straight_1x02_Pitch2.54mm, symbol CONN_01X02
- added J5: Q_QNOT_LATCHED, Pin_Headers:Pin_Header_Straight_1x02_Pitch2.54mm, symbol CONN_01X02
- C3: footprint Capacitors_ThroughHole:CP_Radial_D5.0mm_P2.00mm -> Capacitors_ThroughHole:CP_Radial_D6.3mm_P2.50mm
- C5, C6, C7: footprint (none) -> Capacitors_SMD:C_0805_HandSoldering
- SW1: footprint (none) -> Pin_Headers:Pin_Header_Straight_1x02_Pitch2.54mm
- U1: footprint Housings_SSOP:TSSOP-14_4.4x5mm_Pitch0.65mm -> SMD_Packages:SSOP-14
- U3: footprint Housings_SSOP:TSSOP-8_3x3mm_Pitch0.65mm -> Housings_SSOP:VSSOP-8_2.3x2mm_Pitch0.5mm
Connections:
- net +12V: now also J4.1 (P1)
- net +5V: now also J1.1 (P1), J2.1 (P1), J3.1 (P1)
- net BSPD_Latched_Output: now also U3.5 (Q), J5.1 (P1); no longer U3.3 (~Q)
- net Current_L: now also J2.2 (P2)
- net Current_R: now also J1.2 (P2)
- net GND: now also J1.3 (P3), J2.3 (P3), J3.3 (P3), J4.2 (P2)
- net Hard_Braking: now also J3.2 (P2)
- new net BSPD_Latched_Output_NOT: J5.2 (P2), U3.3 (~Q)
- no-connect marks 2 -> 1
Other:
- moved on the sheet: R3, R4
