File: Harness/file58B1642D.sch (KiCad schematic (older format))
At the start: 37 parts, among them J10 Conn_01x03, J11 Conn_01x12, J12 Conn_01x12, Q4 Q_PMOS_GSD, Q6 Q_NMOS_GSD, U16 TLP291-4, U19 RI-0505S, U20 ISO1540, U21 TCMT1103, U23 PC_RLY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

Commit message: Fleshed out harness diagram
Changed lines of the file:
@@
 $Descr B 17000 11000
 encoding utf-8
-Sheet 6 6
+Sheet 6 9
 Title "Vehicle Controller"
 Date "2017-03-11"
@@
 	10350 1000 10350 1100
 Wire Wire Line
-	10250 1000 10350 1000
-Wire Wire Line
-	10350 1000 10450 1000
+	10250 1000 10450 1000
 Wire Wire Line
 	9100 6900 9100 6800
@@
 	6650 5150 6650 5100
 Wire Wire Line
-	8300 950  8400 950
-Wire Wire Line
-	8400 950  8800 950
+	8300 950  8800 950
 Wire Wire Line
 	8400 1050 8400 950
@@
 	7850 6550 7750 6550
 Wire Wire Line
-	7850 6250 7850 6300
-Wire Wire Line
-	7850 6300 7850 6550
-Wire Wire Line
-	7850 6300 8000 6300
-Wire Wire Line
-	8000 6300 8300 6300
+	7850 6250 7850 6550
+Wire Wire Line
+	7850 6300 8300 6300
 Wire Wire Line
 	8000 6300 8000 6350
 Connection ~ 7850 6300
 Wire Wire Line
-	7750 6650 8000 6650
-Wire Wire Line
-	8000 6650 8850 6650
+	7750 6650 8850 6650
 Wire Wire Line
 	8000 6650 8000 6550
 Connection ~ 8000 6650
 Wire Wire Line
-	7750 6750 8300 6750
-Wire Wire Line
-	8300 6750 8850 6750
+	7750 6750 8850 6750
 Wire Wire Line
 	8300 6300 8300 6350
@@
 	7900 5100 7900 5200
 Wire Wire Line
-	7800 5200 7900 5200
-Wire Wire Line
-	7900 5200 8100 5200
-Wire Wire Line
-	8100 5200 8550 5200
+	7800 5200 8550 5200
 Wire Wire Line
 	7800 5300 7900 5300
 Wire Wire Line
-	7900 5300 7900 5500
-Wire Wire Line
-	7900 5500 7900 5550
-Wire Wire Line
-	10750 5500 10750 5600
-Wire Wire Line
-	10750 5600 10750 5700
+	7900 5300 7900 5550
+Wire Wire Line
+	10750 5500 10750 5700
 Wire Wire Line
 	10750 5600 11500 5600
@@
 	10950 5800 11500 5800
 Wire Wire Line
-	10750 6000 10950 6000
-Wire Wire Line
-	10950 6000 11500 6000
-Wire Wire Line
-	10750 5900 10750 6000
-Wire Wire Line
-	10750 6000 10750 6100
+	10750 6000 11500 6000
+Wire Wire Line
+	10750 5900 10750 6100
 Wire Wire Line
 	10950 5900 11500 5900
@@
 	12500 5700 12900 5700
 Wire Wire Line
-	6800 5050 6800 5100
-Wire Wire Line
-	6800 5100 6800 5200
-Wire Wire Line
-	6800 5300 6800 5400
-Wire Wire Line
-	6800 5400 6800 5450
-Wire Wire Line
-	6050 6650 6300 6650
-Wire Wire Line
-	6300 6650 6850 6650
-Wire Wire Line
-	6050 6750 6600 6750
-Wire Wire Line
-	6600 6750 6850 6750
-Wire Wire Line
-	6750 6200 6750 6300
-Wire Wire Line
-	6750 6300 6750 6550
+	6800 5050 6800 5200
+Wire Wire Line
+	6800 5300 6800 5450
+Wire Wire Line
+	6050 6650 6850 6650
+Wire Wire Line
+	6050 6750 6850 6750
+Wire Wire Line
+	6750 6200 6750 6550
 Wire Wire Line
 	6300 6350 6300 6300
 Wire Wire Line
-	6300 6300 6600 6300
-Wire Wire Line
-	6600 6300 6750 6300
+	6300 6300 6750 6300
 Connection ~ 6750 6300
 Wire Wire Line
@@
 Connection ~ 6600 6750
 Wire Wire Line
-	12150 3450 12300 3450
-Wire Wire Line
-	12300 3450 12650 3450
+	12150 3450 12650 3450
 Wire Wire Line
 	12400 4050 12150 4050
@@
 	11650 4550 11550 4550
 Wire Wire Line
-	11550 4450 11550 4550
-Wire Wire Line
-	11550 4550 11550 4650
+	11550 4450 11550 4650
 Wire Wire Line
 	12150 4150 12400 4150
 Wire Wire Line
-	11100 3450 11500 3450
-Wire Wire Line
-	11500 3450 11650 3450
+	11100 3450 11650 3450
 Wire Wire Line
 	12150 4550 12250 4550
 Wire Wire Line
-	12250 4450 12250 4550
-Wire Wire Line
-	12250 4550 12250 4650
+	12250 4450 12250 4650
 Wire Wire Line
 	11650 4150 11400 4150
 Wire Wire Line
-	7200 1400 7200 1450
-Wire Wire Line
-	7200 1450 7200 1500
+	7200 1400 7200 1500
 Wire Wire Line
 	7450 1400 7450 1550
 Wire Wire Line
-	7450 750  8200 750
-Wire Wire Line
-	8200 750  8800 750
+	7450 750  8800 750
 Wire Wire Line
 	7450 750  7450 1000
@@
 	8450 1550 8700 1550
 Wire Wire Line
-	7450 1550 7850 1550
-Wire Wire Line
-	7850 1550 8150 1550
-Wire Wire Line
-	7750 850  7850 850
-Wire Wire Line
-	7850 850  8800 850
+	7450 1550 8150 1550
+Wire Wire Line
+	7750 850  8800 850
 Connection ~ 7850 1550
 Wire Wire Line
@@
 Connection ~ 7200 1450
 Wire Wire Line
-	7200 1900 7200 2000
-Wire Wire Line
-	7200 2000 7200 2100
+	7200 1900 7200 2100
 Wire Wire Line
 	6850 1750 6850 1700
 Wire Wire Line
-	6550 1700 6850 1700
-Wire Wire Line
-	6850 1700 6900 1700
+	6550 1700 6900 1700
 Wire Wire Line
 	6850 1950 6850 2000
@@
 Connection ~ 6850 1700
 Wire Wire Line
-	11500 3450 11500 3550
-Wire Wire Line
-	11500 3550 11500 3650
-Wire Wire Line
-	11500 3650 11500 3750
-Wire Wire Line
-	11500 3750 11500 3850
-Wire Wire Line
-	11500 3850 11500 3950
+	11500 3450 11500 3950
 Connection ~ 11500 3550
 Connection ~ 11500 3450
@@
 Connection ~ 11500 3750
 Wire Wire Line
-	12300 3450 12300 3550
-Wire Wire Line
-	12300 3550 12300 3650
-Wire Wire Line
-	12300 3650 12300 3750
-Wire Wire Line
-	12300 3750 12300 3850
-Wire Wire Line
-	12300 3850 12300 3950
+	12300 3450 12300 3950
 Connection ~ 12300 3550
 Connection ~ 12300 3450
@@
 	7700 8100 7700 8200
 Wire Wire Line
-	7600 7900 7700 7900
-Wire Wire Line
-	7700 7900 8250 7900
+	7600 7900 8250 7900
 Wire Wire Line
 	7700 7800 7700 7900
@@
 	6700 7900 7000 7900
 Wire Wire Line
-	5750 7900 5900 7900
-Wire Wire Line
-	5900 7900 6000 7900
+	5750 7900 6000 7900
 Wire Wire Line
 	6400 7900 6500 7900
@@
 	6150 8300 6200 8300
 Wire Wire Line
-	6200 8200 6200 8300
-Wire Wire Line
-	6200 8300 6200 8600
+	6200 8200 6200 8600
 Wire Wire Line
 	5950 8300 5900 8300
@@
 	7600 8850 7700 8850
 Wire Wire Line
-	7700 8850 7700 9250
-Wire Wire Line
-	7700 9250 7700 9650
-Wire Wire Line
-	7700 9650 7700 10050
-Wire Wire Line
-	7700 10050 7700 10150
+	7700 8850 7700 10150
 Wire Wire Line
 	7600 9250 7700 9250
@@
 	7000 8850 6900 8850
 Wire Wire Line
-	6900 8850 6900 9250
-Wire Wire Line
-	6900 9250 6900 9650
-Wire Wire Line
-	6900 9650 6900 10050
-Wire Wire Line
-	6900 10050 6900 10150
+	6900 8850 6900 10150
 Wire Wire Line
 	6900 10050 7000 10050
@@
 	7000 750  7200 750
 Wire Wire Line
-	7200 750  7200 950
-Wire Wire Line
-	7200 950  7200 1000
+	7200 750  7200 1000
 Connection ~ 7200 950
 Wire Wire Line
